Commit message: Dual arm xacro update
xacro to urdf file update

File: DualArm/dualarm_description/urdf/dual_arm.urdf (robot description, URDF)
Before this commit: robot dualarm, 16 links, 15 joints
Links:
- link link_01: mass 6.6152 -> 11.91
- link link_02: mass 8.2662 -> 9.901
- link link_03: mass 2.8163 -> 3.35
- link link_04: mass 3.213 -> 3.51
- link link_05: mass 2.4856 -> 2.59
- link link_06: mass 1.8893 -> 2.49
- link link_07: mass 1.8666 -> 1.86; geometry collision cylinder length=0.235 radius=0.05; visual mesh filename=package://dualarm_description/meshes/dualarm/r_arm5.STL scale=0.001 0.001 0.001
- link link_08: mass 0.0646 -> 2.676
- link link_09: mass 2.8163 -> 3.35
- link link_10: mass 3.213 -> 3.51
- link link_11: mass 2.4856 -> 2.59
- link link_12: mass 1.8893 -> 2.49
- link link_13: mass 1.8666 -> 1.86
Joints:
- removed joint base_link_link_01
- removed joint link_01_link_02
- removed joint link_02_link_03
- removed joint link_02_link_09
- removed joint link_03_link_04
- removed joint link_04_link_05
- removed joint link_05_link_06
- removed joint link_06_link_07
- removed joint link_07_link_08
- removed joint link_09_link_10
- removed joint link_10_link_11
- removed joint link_11_link_12
- removed joint link_12_link_13
- removed joint link_13_link_14
- added joint dualarm_joint1: type revolute, parent base_link, child link_01, origin xyz=0 0 0.352 rpy=0 0 0, axis 0 0 1, limit lower=-1.5708 upper=1.5708 effort=100 velocity=1
- added joint dualarm_joint10: type revolute, parent link_09, child link_10, origin xyz=0 -0.09 0.083 rpy=0 0 0, axis 0 -1 0, limit lower=-1.5708 upper=0.7854 effort=100 velocity=1
- added joint dualarm_joint11: type revolute, parent link_10, child link_11, origin xyz=0 -0.11 0 rpy=0 0 0, axis 1 0 0, limit lower=-1.5708 upper=0.349 effort=100 velocity=1
- added joint dualarm_joint12: type revolute, parent link_11, child link_12, origin xyz=0 0 -0.242 rpy=0 0 0, axis 0 0 1, limit lower=-1.5708 upper=1.5708 effort=100 velocity=1
- added joint dualarm_joint13: type revolute, parent link_12, child link_13, origin xyz=-0.0245 -0.00175 -0.158 rpy=0 0 0, axis 0 -1 0, limit lower=0 upper=2.3562 effort=100 velocity=1
- added joint dualarm_joint14: type revolute, parent link_13, child link_14, origin xyz=0.0245 0.00175 -0.235 rpy=0 0 0, axis 0 0 1, limit lower=-0.7854 upper=0.7854 effort=100 velocity=1
- added joint dualarm_joint2: type revolute, parent link_01, child link_02, origin xyz=0 0 0.148 rpy=0 0 0, axis 0 -1 0, limit lower=-0.2618 upper=1.22173 effort=100 velocity=1
- added joint dualarm_joint3: type revolute, parent link_02, child link_03, origin xyz=0 0.125 0.217 rpy=0 0 0, axis 0 0 -1, limit lower=-1.5708 upper=0.5236 effort=100 velocity=1
- added joint dualarm_joint4: type revolute, parent link_03, child link_04, origin xyz=0 0.1 0.083 rpy=0 0 0, axis 0 1 0, limit lower=-1.5708 upper=0.7854 effort=100 velocity=1
- added joint dualarm_joint5: type revolute, parent link_04, child link_05, origin xyz=0 0.11 0 rpy=0 0 0, axis 1 0 0, limit lower=-1.5708 upper=0.349 effort=100 velocity=1
- added joint dualarm_joint6: type revolute, parent link_05, child link_06, origin xyz=0 0 -0.242 rpy=0 0 0, axis 0 0 1, limit lower=-1.5708 upper=1.5708 effort=100 velocity=0
- added joint dualarm_joint7: type revolute, parent link_06, child link_07, origin xyz=-0.0245 0.00175 -0.158 rpy=0 0 0, axis 0 1 0, limit lower=0 upper=2.3562 effort=100 velocity=1
- added joint dualarm_joint8: type revolute, parent link_07, child link_08, origin xyz=0.0245 -0.00175 -0.235 rpy=0 0 0, axis 0 0 1, limit lower=-1.5708 upper=1.5708 effort=100 velocity=1
- added joint dualarm_joint9: type revolute, parent link_02, child link_09, origin xyz=0 -0.125 0.217 rpy=0 0 0, axis 0 0 -1, limit lower=-1.5708 upper=0.5236 effort=100 velocity=1
- joint base_joint: origin (none) -> xyz=0 0 0 rpy=0 0 0

File: DualArm/dualarm_description/urdf/dual_arm.xacro (robot description, xacro)
@@ -19,11 +19,14 @@
 		origin_xyz="0 0 .176"
 		ixx="${base_link_ixx}" ixy="${base_link_ixy}" ixz="${base_link_ixz}" iyy="${base_link_iyy}" iyz="${base_link_iyz}" izz="${base_link_izz}"
-		colvis_rpy="0 0 0" colvis_xyz="0 0 0.176"
+		col_rpy="0 0 0" col_xyz="0 0 0.176"
+		vis_rpy="0 0 0" vis_xyz="0 0 0.176"
 		radius="0.15"
 		length="${base_link_length}"
+		mesh_file="package://dualarm_description/meshes/dualarm/base.STL"
+		mesh_scale="0.001 0.001 0.001"
 />
 <!-- waist part -->
 <m_joint_100
-		name="${base_link_name}_${waist_link_01_name}"
+		name="dualarm_joint1"
 		type="revolute"
 		axis_xyz="0 0 1"
@@ -40,12 +43,15 @@
 		origin_xyz="0 0 0.1110776"
 		ixx="${waist_link_01_ixx}" ixy="${waist_link_01_ixy}" ixz="${waist_link_01_ixz}" iyy="${waist_link_01_iyy}" iyz="${waist_link_01_iyz}" izz="${waist_link_01_izz}"
-		colvis_rpy="-1.57 0 0" colvis_xyz="0 0 0.1110776"
+		col_rpy="-1.57 0 0" col_xyz="0 0 0.1110776"
+		vis_rpy="0 0 0" vis_xyz="0 0 0.150"
 		radius="0.06"
 		length="${waist_link_01_length}"
-/>
-<m_joint_100
-		name="${waist_link_01_name}_${waist_link_02_name}"
-		type="revolute"
-		axis_xyz="0 1 0"
+		mesh_file="package://dualarm_description/meshes/dualarm/waist_1.STL"
+		mesh_scale="0.001 0.001 0.001"
+/>
+<m_joint_100
+		name="dualarm_joint2"
+		type="revolute"
+		axis_xyz="0 -1 0"
 		origin_rpy="0 0 0"
 		origin_xyz="0 0 0.148"
@@ -60,7 +66,10 @@
 		origin_xyz="0 0 0.1436171"
 		ixx="${waist_link_02_ixx}" ixy="${waist_link_02_ixy}" ixz="${waist_link_02_ixz}" iyy="${waist_link_02_iyy}" iyz="${waist_link_02_iyz}" izz="${waist_link_02_izz}"
-		colvis_rpy="0 0 0" colvis_xyz="0 0 0.1436171"
+		col_rpy="-1.57 0 0" col_xyz="0 0 0.1436171"
+		vis_rpy="0 0 0" vis_xyz="0 0 0"
 		radius="0.2"
 		length="${waist_link_02_length}"
+		mesh_file="package://dualarm_description/meshes/dualarm/waist_2.STL"
+		mesh_scale="0.001 0.001 0.001"
 />
 <!-- right_arm part -->
@@ -71,12 +80,15 @@
 		origin_xyz="0.0002952 0.0341703 0.076461"
 		ixx="${r_arm_link_01_ixx}" ixy="${r_arm_link_01_ixy}" ixz="${r_arm_link_01_ixz}" iyy="${r_arm_link_01_iyy}" iyz="${r_arm_link_01_iyz}" izz="${r_arm_link_01_izz}"
-		colvis_rpy="-1.57 0 0" colvis_xyz="0.0002952 0.0341703 0.076461"
+		col_rpy="0 0 0" col_xyz="0.0002952 0.0341703 0.076461"
+		vis_rpy="0 0 0" vis_xyz="0 0.08 0.083"
 		radius="0.04"
 		length="${r_arm_link_01_length}"
-/>
-<m_joint_100
-		name="${waist_link_02_name}_${r_arm_link_01_name}"
-		type="revolute"
-		axis_xyz="0 0 1"
+		mesh_file="package://dualarm_description/meshes/dualarm/r_arm1.STL"
+		mesh_scale="0.001 0.001 0.001"
+/>
+<m_joint_100
+		name="dualarm_joint3"
+		type="revolute"
+		axis_xyz="0 0 -1"
 		origin_rpy="0 0 0"
 		origin_xyz="0 0.125 0.217"
@@ -91,10 +103,13 @@
 		origin_xyz="0.0112502 0.0950175 0"
 		ixx="${r_arm_link_02_ixx}" ixy="${r_arm_link_02_ixy}" ixz="${r_arm_link_02_ixz}" iyy="${r_arm_link_02_iyy}" iyz="${r_arm_link_02_iyz}" izz="${r_arm_link_02_izz}"
-		colvis_rpy="0 1.57 0" colvis_xyz="0.0112502 0.0950175 0"
+		col_rpy="0 1.57 0" col_xyz="0.0112502 0.0950175 0"
+		vis_rpy="0 0 0" vis_xyz="0 0.11 0"
 		radius="0.04"
 		length="${r_arm_link_02_length}"
-/>
-<m_joint_100
-		name="${r_arm_link_01_name}_${r_arm_link_02_name}"
+		mesh_file="package://dualarm_description/meshes/dualarm/r_arm2.STL"
+		mesh_scale="0.001 0.001 0.001"
+/>
+<m_joint_100
+		name="dualarm_joint4"
 		type="revolute"
 		axis_xyz="0 1 0"
@@ -102,5 +117,6 @@
 		origin_xyz="0 0.1 0.083"
 		parent="${r_arm_link_01_name}"
-		child="${r_arm_link_02_name}" limit_e="100" limit_l="-1.5708" limit_u="0.7854" limit_v="1"
+		child="${r_arm_link_02_name}"
+		limit_e="100" limit_l="-1.5708" limit_u="0.7854" limit_v="1"
 />
 <m_link_cylinder
@@ -110,12 +126,15 @@
 		origin_xyz="0.0015675 0.0003615 -0.1633768"
 		ixx="${r_arm_link_03_ixx}" ixy="${r_arm_link_03_ixy}" ixz="${r_arm_link_03_ixz}" iyy="${r_arm_link_03_iyy}" iyz="${r_arm_link_03_iyz}" izz="${r_arm_link_03_izz}"
-		colvis_rpy="3.14 0 0" colvis_xyz="0.0015675 0.0003615 -0.1633768"
+		col_rpy="3.14 0 0" col_xyz="0.0015675 0.0003615 -0.1633768"
+		vis_rpy="0 0 0" vis_xyz="0 0 -0.242"
 		radius="0.05"
 		length="${r_arm_link_03_length}"
-/>
-<m_joint_100
-		name="${r_arm_link_02_name}_${r_arm_link_03_name}"
-		type="revolute"
-		axis_xyz="-1 0 0"
+		mesh_file="package://dualarm_description/meshes/dualarm/r_arm3.STL"
+		mesh_scale="0.001 0.001 0.001"
+/>
+<m_joint_100
+		name="dualarm_joint5"
+		type="revolute"
+		axis_xyz="1 0 0"
 		origin_rpy="0 0 0"
 		origin_xyz="0 0.11 0"
@@ -130,25 +149,207 @@
 		origin_xyz="0.0219475 -0.008888 -0.1347982"
 		ixx="${r_arm_link_04_ixx}" ixy="${r_arm_link_04_ixy}" ixz="${r_arm_link_04_ixz}" iyy="${r_arm_link_04_iyy}" iyz="${r_arm_link_04_iyz}" izz="${r_arm_link_04_izz}"
-		colvis_rpy="1.57 0 0" colvis_xyz="0.0219475 -0.008888 -0.1347982"
+		col_rpy="1.57 0 0" col_xyz="0.0219475 -0.008888 -0.1347982"
+		vis_rpy="0 0 0" vis_xyz="-0.00245 0.00175 -0.158"
 		radius="0.05"
 		length="${r_arm_link_04_length}"
-/>
-<m_joint_100 name="${r_arm_link_03_name}_${r_arm_link_04_name}" type="revolute" axis_xyz="0 0 1" origin_rpy="0 0 0" origin_xyz="0 0 -0.242" parent="${r_arm_link_03_name}" child="${r_arm_link_04_name}" limit_e="100" limit_l="-1.5708" limit_u="1.5708" limit_v="0"/>
-<m_link_cylinder name="${r_arm_link_05_name}" mass="${r_arm_link_05_mass}" origin_rpy="0 0 0" origin_xyz="0.0282566 -0.0026831 -0.1626786" ixx="${r_arm_link_05_ixx}" ixy="${r_arm_link_05_ixy}" ixz="${r_arm_link_05_ixz}" iyy="${r_arm_link_05_iyy}" iyz="${r_arm_link_05_iyz}" izz="${r_arm_link_05_izz}" colvis_rpy="0 0 0" colvis_xyz="0.0282566 -0.0026831 -0.1626786" radius="0.05" length="0.158"/>
-<m_joint_100 name="${r_arm_link_04_name}_${r_arm_link_05_name}" type="revolute" axis_xyz="0 -1 0" origin_rpy="0 0 0" origin_xyz="-0.0245 0.00175 -0.158" parent="${r_arm_link_04_name}" child="${r_arm_link_05_name}" limit_e="100" limit_l="0" limit_u="2.3562" limit_v="1"/>
-<m_link_cylinder name="${r_arm_link_06_name}" mass="${r_arm_link_06_mass}" origin_rpy="0 0 0" origin_xyz="0 -0.0027174 -0.0051051" ixx="${r_arm_link_06_ixx}" ixy="${r_arm_link_06_ixy}" ixz="${r_arm_link_06_ixz}" iyy="${r_arm_link_06_iyy}" iyz="${r_arm_link_06_iyz}" izz="${r_arm_link_06_izz}" colvis_rpy="0 0 0" colvis_xyz="0 -0.0027174 -0.0051051" radius="0.05" length="${r_arm_link_06_length}"/>
-<m_joint_100 name="${r_arm_link_05_name}_${r_arm_link_06_name}" type="revolute" axis_xyz="0 0 1" origin_rpy="0 0 0" origin_xyz="0.0245 -0.00175 -0.235" parent="${r_arm_link_05_name}" child="${r_arm_link_06_name}" limit_e="100" limit_l="-0.7854" limit_u="0.7854" limit_v="0"/>
+		mesh_file="package://dualarm_description/meshes/dualarm/r_arm4.STL"
+		mesh_scale="0.001 0.001 0.001"
+/>
+<m_joint_100
+		name="dualarm_joint6"
+		type="revolute"
+		axis_xyz="0 0 1"
+		origin_rpy="0 0 0"
+		origin_xyz="0 0 -0.242"
+		parent="${r_arm_link_03_name}"
+		child="${r_arm_link_04_name}"
+		limit_e="100" limit_l="-1.5708" limit_u="1.5708" limit_v="0"
+/>
+<m_link_cylinder
+		name="${r_arm_link_05_name}"
+		mass="${r_arm_link_05_mass}"
+		origin_rpy="0 0 0"
+		origin_xyz="0.0282566 -0.0026831 -0.1626786"
+		ixx="${r_arm_link_05_ixx}" ixy="${r_arm_link_05_ixy}" ixz="${r_arm_link_05_ixz}" iyy="${r_arm_link_05_iyy}" iyz="${r_arm_link_05_iyz}" izz="${r_arm_link_05_izz}"
+		col_rpy="0 0 0" col_xyz="0.0282566 -0.0026831 -0.1626786"
+		vis_rpy="0 0 0" vis_xyz="0 0 0"
+		radius="0.05"
+		length="${r_arm_link_05_length}"
+		mesh_file="package://dualarm_description/meshes/dualarm/r_arm5.STL"
+		mesh_scale="0.001 0.001 0.001"
+/>
+<m_joint_100
+		name="dualarm_joint7"
+		type="revolute"
+		axis_xyz="0 1 0"
+		origin_rpy="0 0 0"
+		origin_xyz="-0.0245 0.00175 -0.158"
+		parent="${r_arm_link_04_name}"
+		child="${r_arm_link_05_name}"
+		limit_e="100" limit_l="0" limit_u="2.3562" limit_v="1"
+/>
+<m_link_cylinder
+		name="${r_arm_link_06_name}"
+		mass="${r_arm_link_06_mass}"
+		origin_rpy="0 0 0"
+		origin_xyz="0 -0.0027174 -0.0051051"
+		ixx="${r_arm_link_06_ixx}" ixy="${r_arm_link_06_ixy}" ixz="${r_arm_link_06_ixz}" iyy="${r_arm_link_06_iyy}" iyz="${r_arm_link_06_iyz}" izz="${r_arm_link_06_izz}"
+		col_rpy="0 0 0" col_xyz="0 -0.0027174 -0.0051051"
+		vis_rpy="3.14 0 0" vis_xyz="-0.032 0.034 0.085"
+		radius="0.05"
+		length="${r_arm_link_06_length}"
+		mesh_file="package://dualarm_description/meshes/dualarm/link6.STL"
+		mesh_scale="0.001 0.001 0.001"
+/>
+<m_joint_100
+		name="dualarm_joint8"
+		type="revolute"
+		axis_xyz="0 0 1"
+		origin_rpy="0 0 0"
+		origin_xyz="0.0245 -0.00175 -0.235"
+		parent="${r_arm_link_05_name}"
+		child="${r_arm_link_06_name}"
+		limit_e="100" limit_l="-1.5708" limit_u="1.5708" limit_v="1"
+/>
 <!-- left_arm part-->
-<m_link_cylinder name="${l_arm_link_01_name}" mass="${l_arm_link_01_mass}" origin_rpy="0 0 0" origin_xyz="0.0002952 -0.0341703 0.076461" ixx="${l_arm_link_01_ixx}" ixy="${l_arm_link_01_ixy}" ixz="${l_arm_link_01_ixz}" iyy="${l_arm_link_01_iyy}" iyz="${l_arm_link_01_iyz}" izz="${l_arm_link_01_izz}" colvis_rpy="1.57 0 0" colvis_xyz="0.0002952 -0.0341703 0.076461" radius="0.04" length="${l_arm_link_01_length}"/>
-<m_joint_100 name="${waist_link_02_name}_${l_arm_link_01_name}" type="revolute" axis_xyz="0 0 -1" origin_rpy="0 0 0" origin_xyz="0 -0.125 0.217" parent="${waist_link_02_name}" child="${l_arm_link_01_name}" limit_e="100" limit_l="-1.5708" limit_u="0.5236" limit_v="1"/>
-<m_link_cylinder name="${l_arm_link_02_name}" mass="${l_arm_link_02_mass}" origin_rpy="0 0 0" origin_xyz="0.0112502 -0.0950175 0" ixx="${l_arm_link_02_ixx}" ixy="${l_arm_link_02_ixy}" ixz="${l_arm_link_02_ixz}" iyy="${l_arm_link_02_iyy}" iyz="${l_arm_link_02_iyz}" izz="${l_arm_link_02_izz}" colvis_rpy="0 -1.57 0" colvis_xyz="0.0112502 -0.0950175 0" radius="0.04" length="${l_arm_link_02_length}"/>
-<m_joint_100 name="${l_arm_link_01_name}_${l_arm_link_02_name}" type="revolute" axis_xyz="0 -1 0" origin_rpy="0 0 0" origin_xyz="0 -0.09 0.083" parent="${l_arm_link_01_name}" child="${l_arm_link_02_name}" limit_e="100" limit_l="-1.5708" limit_u="0.7854" limit_v="1"/>
-<m_link_cylinder name="${l_arm_link_03_name}" mass="${l_arm_link_03_mass}" origin_rpy="0 0 0" origin_xyz="0.0015675 -0.0003615 -0.1633768" ixx="${l_arm_link_03_ixx}" ixy="${l_arm_link_03_ixy}" ixz="${l_arm_link_03_ixz}" iyy="${l_arm_link_03_iyy}" iyz="${l_arm_link_03_iyz}" izz="${l_arm_link_03_izz}" colvis_rpy="0 0 0" colvis_xyz="0.0015675 -0.0003615 -0.1633768" radius="0.05" length="${l_arm_link_03_length}"/>
-<m_joint_100 name="${l_arm_link_02_name}_${l_arm_link_03_name}" type="revolute" axis_xyz="1 0 0" origin_rpy="0 0 0" origin_xyz="0 -0.11 0" parent="${l_arm_link_02_name}" child="${l_arm_link_03_name}" limit_e="100" limit_l="-1.5708" limit_u="0.3490" limit_v="1"/>
-<m_link_cylinder name="${l_arm_link_04_name}" mass="${l_arm_link_04_mass}" origin_rpy="0 0 0" origin_xyz="0.0219475 0.008888 -0.1347982" ixx="${l_arm_link_04_ixx}" ixy="${l_arm_link_04_ixy}" ixz="${l_arm_link_04_ixz}" iyy="${l_arm_link_04_iyy}" iyz="${l_arm_link_04_iyz}" izz="${l_arm_link_04_izz}" colvis_rpy="-1.57 0 0" colvis_xyz="0.0219475 0.008888 -0.1347982" radius="0.05" length="${l_arm_link_04_length}"/>
-<m_joint_100 name="${l_arm_link_03_name}_${l_arm_link_04_name}" type="revolute" axis_xyz="0 0 -1" origin_rpy="0 0 0" origin_xyz="0 0 -0.242" parent="${l_arm_link_03_name}" child="${l_arm_link_04_name}" limit_e="100" limit_l="-1.5708" limit_u="1.5708" limit_v="1"/>
-<m_link_cylinder name="${l_arm_link_05_name}" mass="${l_arm_link_05_mass}" origin_rpy="0 0 0" origin_xyz="0.0282566 0.0026831 -0.1626786" ixx="${l_arm_link_05_ixx}" ixy="${l_arm_link_05_ixy}" ixz="${l_arm_link_05_ixz}" iyy="${l_arm_link_05_iyy}" iyz="${l_arm_link_05_iyz}" izz="${l_arm_link_05_izz}" colvis_rpy="0 0 0" colvis_xyz="0.0282566 0.0026831 -0.1626786" radius="0.05" length="0.158"/>
-<m_joint_100 name="${l_arm_link_04_name}_${l_arm_link_05_name}" type="revolute" axis_xyz="0 -1 0" origin_rpy="0 0 0" origin_xyz="-0.0245 -0.00175 -0.158" parent="${l_arm_link_04_name}" child="${l_arm_link_05_name}" limit_e="100" limit_l="0" limit_u="2.3562" limit_v="1"/>
-<m_link_cylinder name="${l_arm_link_06_name}" mass="${l_arm_link_06_mass}" origin_rpy="0 0 0" origin_xyz="0 0.0027174 -0.0051051" ixx="${l_arm_link_06_ixx}" ixy="${l_arm_link_06_ixy}" ixz="${l_arm_link_06_ixz}" iyy="${l_arm_link_06_iyy}" iyz="${l_arm_link_06_iyz}" izz="${l_arm_link_06_izz}" colvis_rpy="0 0 0" colvis_xyz="0 0.0027174 -0.0051051" radius="0.05" length="${l_arm_link_06_length}"/>
-<m_joint_100 name="${l_arm_link_05_name}_${l_arm_link_06_name}" type="revolute" axis_xyz="0 0 -1" origin_rpy="0 0 0" origin_xyz="0.0245 0.00175 -0.235" parent="${l_arm_link_05_name}" child="${l_arm_link_06_name}" limit_e="100" limit_l="-0.7854" limit_u="0.7854" limit_v="1"/>
+<m_link_cylinder
+		name="${l_arm_link_01_name}"
+		mass="${l_arm_link_01_mass}"
+		origin_rpy="0 0 0"
+		origin_xyz="0.0002952 -0.0341703 0.076461"
+		ixx="${l_arm_link_01_ixx}"
+		ixy="${l_arm_link_01_ixy}"
+		ixz="${l_arm_link_01_ixz}" iyy="${l_arm_link_01_iyy}" iyz="${l_arm_link_01_iyz}" izz="${l_arm_link_01_izz}"
+		col_rpy="1.57 0 0" col_xyz="0.0002952 -0.0341703 0.076461"
+		vis_rpy="0 0 0" vis_xyz="0 -0.075 0.083"
+		radius="0.04"
+		length="${l_arm_link_01_length}"
+		mesh_file="package://dualarm_description/meshes/dualarm/l_arm1.STL"
+		mesh_scale="0.001 0.001 0.001"
+/>
+<m_joint_100
+		name="dualarm_joint9"
+		type="revolute"
+		axis_xyz="0 0 -1"
+		origin_rpy="0 0 0"
+		origin_xyz="0 -0.125 0.217"
+		parent="${waist_link_02_name}"
+		child="${l_arm_link_01_name}"
+		limit_e="100" limit_l="-1.5708" limit_u="0.5236" limit_v="1"
+/>
+<m_link_cylinder
+		name="${l_arm_link_02_name}"
+		mass="${l_arm_link_02_mass}"
+		origin_rpy="0 0 0"
+		origin_xyz="0.0112502 -0.0950175 0"
+		ixx="${l_arm_link_02_ixx}" ixy="${l_arm_link_02_ixy}" ixz="${l_arm_link_02_ixz}" iyy="${l_arm_link_02_iyy}" iyz="${l_arm_link_02_iyz}" izz="${l_arm_link_02_izz}"
+		col_rpy="0 -1.57 0" col_xyz="0.0112502 -0.0950175 0"
+		vis_rpy="0 0 0" vis_xyz="0 -0.11 -0.00"
+		radius="0.04"
+		length="${l_arm_link_02_length}"
+		mesh_file="package://dualarm_description/meshes/dualarm/l_arm2.STL"
+		mesh_scale="0.001 0.001 0.001"
+/>
+<m_joint_100
+		name="dualarm_joint10"
+		type="revolute"
+		axis_xyz="0 -1 0"
+		origin_rpy="0 0 0"
+		origin_xyz="0 -0.09 0.083"
+		parent="${l_arm_link_01_name}"
+		child="${l_arm_link_02_name}"
+		limit_e="100" limit_l="-1.5708" limit_u="0.7854" limit_v="1"
+/>
+<m_link_cylinder
+		name="${l_arm_link_03_name}"
+		mass="${l_arm_link_03_mass}"
+		origin_rpy="0 0 0"
+		origin_xyz="0.0015675 -0.0003615 -0.1633768"
+		ixx="${l_arm_link_03_ixx}" ixy="${l_arm_link_03_ixy}" ixz="${l_arm_link_03_ixz}" iyy="${l_arm_link_03_iyy}" iyz="${l_arm_link_03_iyz}" izz="${l_arm_link_03_izz}"
+		col_rpy="0 0 0" col_xyz="0.0015675 -0.0003615 -0.1633768"
+		vis_rpy="0 0 0" vis_xyz="0 0 -0.242"
+		radius="0.05"
+		length="${l_arm_link_03_length}"
+		mesh_file="package://dualarm_description/meshes/dualarm/l_arm3.STL"
+		mesh_scale="0.001 0.001 0.001"
+/>
+<m_joint_100
+		name="dualarm_joint11"
+		type="revolute"
+		axis_xyz="1 0 0"
+		origin_rpy="0 0 0"
+		origin_xyz="0 -0.11 0"
+		parent="${l_arm_link_02_name}"
+		child="${l_arm_link_03_name}"
+		limit_e="100" limit_l="-1.5708" limit_u="0.3490" limit_v="1"
+/>
+<m_link_cylinder
+		name="${l_arm_link_04_name}"
+		mass="${l_arm_link_04_mass}"
+		origin_rpy="0 0 0"
+		origin_xyz="0.0219475 0.008888 -0.1347982"
+		ixx="${l_arm_link_04_ixx}" ixy="${l_arm_link_04_ixy}" ixz="${l_arm_link_04_ixz}" iyy="${l_arm_link_04_iyy}" iyz="${l_arm_link_04_iyz}" izz="${l_arm_link_04_izz}"
+		col_rpy="-1.57 0 0" col_xyz="0.0219475 0.008888 -0.1347982"
+		vis_rpy="0 0 0" vis_xyz="-0.0245 -0.00175 -0.158"
+		radius="0.05"
+		length="${l_arm_link_04_length}"
+		mesh_file="package://dualarm_description/meshes/dualarm/l_arm4.STL"
+		mesh_scale="0.001 0.001 0.001"
+/>
+<m_joint_100
+		name="dualarm_joint12"
+		type="revolute"
+		axis_xyz="0 0 1"
+		origin_rpy="0 0 0"
+		origin_xyz="0 0 -0.242"
+		parent="${l_arm_link_03_name}"
+		child="${l_arm_link_04_name}"
+		limit_e="100" limit_l="-1.5708" limit_u="1.5708" limit_v="1"
+/>
+<m_link_cylinder
+		name="${l_arm_link_05_name}"
+		mass="${l_arm_link_05_mass}"
+		origin_rpy="0 0 0"
+		origin_xyz="0.0282566 0.0026831 -0.1626786"
+		ixx="${l_arm_link_05_ixx}" ixy="${l_arm_link_05_ixy}" ixz="${l_arm_link_05_ixz}" iyy="${l_arm_link_05_iyy}" iyz="${l_arm_link_05_iyz}" izz="${l_arm_link_05_izz}"
+		col_rpy="0 0 0" col_xyz="0.0282566 0.0026831 -0.1626786"
+		vis_rpy="0 0 0" vis_xyz="0 0 0"
+		radius="0.05"
+		length="0.158"
+		mesh_file="package://dualarm_description/meshes/dualarm/l_arm5.STL"
+		mesh_scale="0.001 0.001 0.001"
+/>
+<m_joint_100
+		name="dualarm_joint13"
+		type="revolute"
+		axis_xyz="0 -1 0"
+		origin_rpy="0 0 0"
+		origin_xyz="-0.0245 -0.00175 -0.158"
+		parent="${l_arm_link_04_name}"
+		child="${l_arm_link_05_name}"
+		limit_e="100" limit_l="0" limit_u="2.3562" limit_v="1"
+/>
+<m_link_cylinder
+		name="${l_arm_link_06_name}"
+		mass="${l_arm_link_06_mass}"
+		origin_rpy="0 0 0"
+		origin_xyz="0 0.0027174 -0.0051051"
+		ixx="${l_arm_link_06_ixx}" ixy="${l_arm_link_06_ixy}" ixz="${l_arm_link_06_ixz}" iyy="${l_arm_link_06_iyy}" iyz="${l_arm_link_06_iyz}" izz="${l_arm_link_06_izz}"
+		col_rpy="0 0 0" col_xyz="0 0.0027174 -0.0051051"
+		vis_rpy="3.14 0 0" vis_xyz="-0.032 0.034 0.085"
+		radius="0.05"
+		length="${l_arm_link_06_length}"
+		mesh_file="package://dualarm_description/meshes/dualarm/link6.STL"
+		mesh_scale="0.001 0.001 0.001"
+/>
+<m_joint_100
+		name="dualarm_joint14"
+		type="revolute"
+		axis_xyz="0 0 1"
+		origin_rpy="0 0 0"
+		origin_xyz="0.0245 0.00175 -0.235"
+		parent="${l_arm_link_05_name}"
+		child="${l_arm_link_06_name}"
+		limit_e="100" limit_l="-0.7854" limit_u="0.7854" limit_v="1"
+/>
 </robot>

File: DualArm/dualarm_description/urdf/link_to_joint.xacro (robot description, xacro)
@@ -20,5 +20,6 @@
     </transmission>
   </xacro:macro>
-  <xacro:macro name="m_link_cylinder" params="name origin_xyz origin_rpy colvis_xyz colvis_rpy radius length mass ixx ixy ixz iyy iyz izz">
+  <xacro:macro name="m_link_cylinder"
+               params="name origin_xyz origin_rpy col_xyz col_rpy vis_rpy vis_xyz radius length mass ixx ixy ixz iyy iyz izz mesh_file mesh_scale">
     <link name="${name}">
       <inertial>
@@ -28,5 +29,5 @@
       </inertial>
       <collision>
-        <origin rpy="${colvis_rpy}" xyz="${colvis_xyz}" />
+        <origin rpy="${col_rpy}" xyz="${col_xyz}" />
         <geometry>
           <cylinder radius="${radius}" length="${length}" />
@@ -34,7 +35,7 @@
       </collision>
       <visual>
-        <origin rpy="${colvis_rpy}" xyz="${colvis_xyz}" />
+        <origin rpy="${vis_rpy}" xyz="${vis_xyz}" />
         <geometry>
-          <cylinder radius="${radius}" length="${length}" />
+          <mesh filename="${mesh_file}" scale="${mesh_scale}"/>
         </geometry>
       </visual>
