Commit message: CLIK update
update check

File: DualArm/dualarm_description/urdf/dual_arm.urdf (robot description, URDF)
Before this commit: robot dualarm, 16 links, 15 joints
Links:
- added link dual_arm_base_link
- link base_link: geometry visual mesh filename=package://dualarm_description/meshes/dualarm/base.STL scale=0.001 0.001 0.001
- link link_01: geometry visual mesh filename=package://dualarm_description/meshes/dualarm/waist_1.STL scale=0.001 0.001 0.001
- link link_02: geometry visual mesh filename=package://dualarm_description/meshes/dualarm/waist_2.STL scale=0.001 0.001 0.001
- link link_03: geometry visual mesh filename=package://dualarm_description/meshes/dualarm/r_arm1.STL scale=0.001 0.001 0.001
- link link_04: geometry visual mesh filename=package://dualarm_description/meshes/dualarm/r_arm2.STL scale=0.001 0.001 0.001
- link link_05: geometry visual mesh filename=package://dualarm_description/meshes/dualarm/r_arm3.STL scale=0.001 0.001 0.001
- link link_06: geometry visual mesh filename=package://dualarm_description/meshes/dualarm/r_arm4.STL scale=0.001 0.001 0.001
- link link_07: geometry visual mesh filename=package://dualarm_description/meshes/dualarm/r_arm5.STL scale=0.001 0.001 0.001
- link link_08: geometry visual mesh filename=package://dualarm_description/meshes/dualarm/link6.STL scale=0.001 0.001 0.001
- link link_09: geometry visual mesh filename=package://dualarm_description/meshes/dualarm/l_arm1.STL scale=0.001 0.001 0.001
- link link_10: geometry visual mesh filename=package://dualarm_description/meshes/dualarm/l_arm2.STL scale=0.001 0.001 0.001
- link link_11: geometry visual mesh filename=package://dualarm_description/meshes/dualarm/l_arm3.STL scale=0.001 0.001 0.001
- link link_12: geometry visual mesh filename=package://dualarm_description/meshes/dualarm/l_arm4.STL scale=0.001 0.001 0.001
- link link_13: geometry visual mesh filename=package://dualarm_description/meshes/dualarm/l_arm5.STL scale=0.001 0.001 0.001
- link link_14: geometry visual mesh filename=package://dualarm_description/meshes/dualarm/link6.STL scale=0.001 0.001 0.001
Joints:
- added joint dual_arm_base_joint: type fixed, parent dual_arm_base_link, child base_link, origin xyz=0 0 0 rpy=0 0 0
- joint base_joint: child base_link -> dual_arm_base_link
- joint dualarm_joint1: limit lower=-1.5708 upper=1.5708 effort=100 velocity=1 -> lower=-1.570795 upper=1.570795 effort=100 velocity=1
- joint dualarm_joint10: limit lower=-1.5708 upper=0.7854 effort=100 velocity=1 -> lower=-1.570795 upper=0.7853975 effort=100 velocity=1; origin xyz=0 -0.09 0.083 rpy=0 0 0 -> xyz=0 0.09 0.083 rpy=0 0 0
- joint dualarm_joint11: limit lower=-1.5708 upper=0.349 effort=100 velocity=1 -> lower=-0.7853975 upper=1.570795 effort=100 velocity=1; origin xyz=0 -0.11 0 rpy=0 0 0 -> xyz=0 0.11 0 rpy=0 0 0
- joint dualarm_joint12: limit lower=-1.5708 upper=1.5708 effort=100 velocity=1 -> lower=-1.570795 upper=1.570795 effort=100 velocity=1; origin xyz=0 0 -0.242 rpy=0 0 0 -> xyz=0 0 -0.158 rpy=0 0 0
- joint dualarm_joint13: limit lower=0 upper=2.3562 effort=100 velocity=1 -> lower=-1.570795 upper=0.7853975 effort=100 velocity=1; origin xyz=-0.0245 -0.00175 -0.158 rpy=0 0 0 -> xyz=-0.0245 0 -0.158 rpy=0 0 0
- joint dualarm_joint14: limit lower=-0.7854 upper=0.7854 effort=100 velocity=1 -> lower=-0.7853975 upper=0.7853975 effort=100 velocity=1; origin xyz=0.0245 0.00175 -0.235 rpy=0 0 0 -> xyz=0.0245 0 -0.155 rpy=0 0 0
- joint dualarm_joint2: axis 0 -1 0 -> 0 1 0; limit lower=-0.2618 upper=1.22173 effort=100 velocity=1 -> lower=1.570795 upper=-0.39269875 effort=100 velocity=1
- joint dualarm_joint3: limit lower=-1.5708 upper=0.5236 effort=100 velocity=1 -> lower=-1.570795 upper=0.7853975 effort=100 velocity=1; origin xyz=0 0.125 0.217 rpy=0 0 0 -> xyz=0 -0.125 0.217 rpy=0 0 0
- joint dualarm_joint4: limit lower=-1.5708 upper=0.7854 effort=100 velocity=1 -> lower=-0.7853975 upper=1.570795 effort=100 velocity=1; origin xyz=0 0.1 0.083 rpy=0 0 0 -> xyz=0 -0.09 0.083 rpy=0 0 0
- joint dualarm_joint5: limit lower=-1.5708 upper=0.349 effort=100 velocity=1 -> lower=-1.570795 upper=0.7853975 effort=100 velocity=1; origin xyz=0 0.11 0 rpy=0 0 0 -> xyz=0 -0.11 0 rpy=0 0 0
- joint dualarm_joint6: limit lower=-1.5708 upper=1.5708 effort=100 velocity=0 -> lower=-1.570795 upper=1.570795 effort=100 velocity=1; origin xyz=0 0 -0.242 rpy=0 0 0 -> xyz=0 0 -0.158 rpy=0 0 0
- joint dualarm_joint7: limit lower=0 upper=2.3562 effort=100 velocity=1 -> lower=-0.39269875 upper=1.570795 effort=100 velocity=1; origin xyz=-0.0245 0.00175 -0.158 rpy=0 0 0 -> xyz=-0.0245 0 -0.158 rpy=0 0 0
- joint dualarm_joint8: limit lower=-1.5708 upper=1.5708 effort=100 velocity=1 -> lower=-0.7853975 upper=0.7853975 effort=100 velocity=1; origin xyz=0.0245 -0.00175 -0.235 rpy=0 0 0 -> xyz=0.0245 0 -0.155 rpy=0 0 0
- joint dualarm_joint9: limit lower=-1.5708 upper=0.5236 effort=100 velocity=1 -> lower=-0.7853975 upper=1.570795 effort=100 velocity=1; origin xyz=0 -0.125 0.217 rpy=0 0 0 -> xyz=0 0.125 0.217 rpy=0 0 0

File: DualArm/dualarm_description/urdf/dual_arm.xacro (robot description, xacro)
@@ -4,352 +4,449 @@
 	<xacro:include filename="$(find dualarm_description)/urdf/robot_parameter.xacro" />
 	<xacro:include filename="$(find dualarm_description)/urdf/dual_arm.gazebo" />
-<!-- Base parts -->
-<link name = "world"/>
-<joint name="base_joint" type="fixed">
-	<origin
-		xyz="0 0 0"
-		rpy="0 0 0"/>
-	<parent link="world"/>
-	<child link="${base_link_name}"/>
-</joint>
-<m_link_cylinder
-		name="${base_link_name}"
-		mass = "${base_link_mass}"
-		origin_rpy = "0 0 0"
-		origin_xyz="0 0 .176"
-		ixx="${base_link_ixx}" ixy="${base_link_ixy}" ixz="${base_link_ixz}" iyy="${base_link_iyy}" iyz="${base_link_iyz}" izz="${base_link_izz}"
-		col_rpy="0 0 0" col_xyz="0 0 0.176"
-		vis_rpy="0 0 0" vis_xyz="0 0 0.176"
-		radius="0.15"
-		length="${base_link_length}"
-		mesh_file="package://dualarm_description/meshes/dualarm/base.STL"
-		mesh_scale="0.001 0.001 0.001"
-/>
-<!-- waist part -->
-<m_joint_100
-		name="dualarm_joint1"
-		type="revolute"
-		axis_xyz="0 0 1"
-		origin_rpy="0 0 0"
-		origin_xyz="0 0 0.352"
-		parent="${base_link_name}"
-		child="${waist_link_01_name}"
-		limit_e="100" limit_l="-1.5708" limit_u="1.5708" limit_v="1"
-/>
-<m_link_cylinder
-		name="${waist_link_01_name}"
-		mass="${waist_link_01_mass}"
-		origin_rpy="0 0 0"
-		origin_xyz="0 0 0.1110776"
-		ixx="${waist_link_01_ixx}" ixy="${waist_link_01_ixy}" ixz="${waist_link_01_ixz}" iyy="${waist_link_01_iyy}" iyz="${waist_link_01_iyz}" izz="${waist_link_01_izz}"
-		col_rpy="-1.57 0 0" col_xyz="0 0 0.1110776"
-		vis_rpy="0 0 0" vis_xyz="0 0 0.150"
-		radius="0.06"
-		length="${waist_link_01_length}"
-		mesh_file="package://dualarm_description/meshes/dualarm/waist_1.STL"
-		mesh_scale="0.001 0.001 0.001"
-/>
-<m_joint_100
-		name="dualarm_joint2"
-		type="revolute"
-		axis_xyz="0 -1 0"
-		origin_rpy="0 0 0"
-		origin_xyz="0 0 0.148"
-		parent="${waist_link_01_name}"
-		child="${waist_link_02_name}"
-		limit_e="100" limit_u="1.22173" limit_l="-0.2618" limit_v="1"
-/>
-<m_link_cylinder
-		name="${waist_link_02_name}"
-		mass="${waist_link_02_mass}"
-		origin_rpy="0 0 0"
-		origin_xyz="0 0 0.1436171"
-		ixx="${waist_link_02_ixx}" ixy="${waist_link_02_ixy}" ixz="${waist_link_02_ixz}" iyy="${waist_link_02_iyy}" iyz="${waist_link_02_iyz}" izz="${waist_link_02_izz}"
-		col_rpy="-1.57 0 0" col_xyz="0 0 0.1436171"
-		vis_rpy="0 0 0" vis_xyz="0 0 0"
-		radius="0.2"
-		length="${waist_link_02_length}"
-		mesh_file="package://dualarm_description/meshes/dualarm/waist_2.STL"
-		mesh_scale="0.001 0.001 0.001"
-/>
-<!-- right_arm part -->
-<m_link_cylinder
-		name="${r_arm_link_01_name}"
-		mass="${r_arm_link_01_mass}"
-		origin_rpy="0 0 0"
-		origin_xyz="0.0002952 0.0341703 0.076461"
-		ixx="${r_arm_link_01_ixx}" ixy="${r_arm_link_01_ixy}" ixz="${r_arm_link_01_ixz}" iyy="${r_arm_link_01_iyy}" iyz="${r_arm_link_01_iyz}" izz="${r_arm_link_01_izz}"
-		col_rpy="0 0 0" col_xyz="0.0002952 0.0341703 0.076461"
-		vis_rpy="0 0 0" vis_xyz="0 0.08 0.083"
-		radius="0.04"
-		length="${r_arm_link_01_length}"
-		mesh_file="package://dualarm_description/meshes/dualarm/r_arm1.STL"
-		mesh_scale="0.001 0.001 0.001"
-/>
-<m_joint_100
-		name="dualarm_joint3"
-		type="revolute"
-		axis_xyz="0 0 -1"
-		origin_rpy="0 0 0"
-		origin_xyz="0 0.125 0.217"
-		parent="${waist_link_02_name}"
-		child="${r_arm_link_01_name}"
-		limit_e="100" limit_l="-1.5708" limit_u="0.5236" limit_v="1"
-/>
-<m_link_cylinder
-		name="${r_arm_link_02_name}"
-		mass="${r_arm_link_02_mass}"
-		origin_rpy="0 0 0"
-		origin_xyz="0.0112502 0.0950175 0"
-		ixx="${r_arm_link_02_ixx}" ixy="${r_arm_link_02_ixy}" ixz="${r_arm_link_02_ixz}" iyy="${r_arm_link_02_iyy}" iyz="${r_arm_link_02_iyz}" izz="${r_arm_link_02_izz}"
-		col_rpy="0 1.57 0" col_xyz="0.0112502 0.0950175 0"
-		vis_rpy="0 0 0" vis_xyz="0 0.11 0"
-		radius="0.04"
-		length="${r_arm_link_02_length}"
-		mesh_file="package://dualarm_description/meshes/dualarm/r_arm2.STL"
-		mesh_scale="0.001 0.001 0.001"
-/>
-<m_joint_100
-		name="dualarm_joint4"
-		type="revolute"
-		axis_xyz="0 1 0"
-		origin_rpy="0 0 0"
-		origin_xyz="0 0.1 0.083"
-		parent="${r_arm_link_01_name}"
-		child="${r_arm_link_02_name}"
-		limit_e="100" limit_l="-1.5708" limit_u="0.7854" limit_v="1"
-/>
-<m_link_cylinder
-		name="${r_arm_link_03_name}"
-		mass="${r_arm_link_03_mass}"
-		origin_rpy="0 0 0"
-		origin_xyz="0.0015675 0.0003615 -0.1633768"
-		ixx="${r_arm_link_03_ixx}" ixy="${r_arm_link_03_ixy}" ixz="${r_arm_link_03_ixz}" iyy="${r_arm_link_03_iyy}" iyz="${r_arm_link_03_iyz}" izz="${r_arm_link_03_izz}"
-		col_rpy="3.14 0 0" col_xyz="0.0015675 0.0003615 -0.1633768"
-		vis_rpy="0 0 0" vis_xyz="0 0 -0.242"
-		radius="0.05"
-		length="${r_arm_link_03_length}"
-		mesh_file="package://dualarm_description/meshes/dualarm/r_arm3.STL"
-		mesh_scale="0.001 0.001 0.001"
-/>
-<m_joint_100
-		name="dualarm_joint5"
-		type="revolute"
-		axis_xyz="1 0 0"
-		origin_rpy="0 0 0"
-		origin_xyz="0 0.11 0"
-		parent="${r_arm_link_02_name}"
-		child="${r_arm_link_03_name}"
-		limit_e="100" limit_l="-1.5708" limit_u="0.3490" limit_v="1"
-/>
-<m_link_cylinder
-		name="${r_arm_link_04_name}"
-		mass="${r_arm_link_04_mass}"
-		origin_rpy="0 0 0"
-		origin_xyz="0.0219475 -0.008888 -0.1347982"
-		ixx="${r_arm_link_04_ixx}" ixy="${r_arm_link_04_ixy}" ixz="${r_arm_link_04_ixz}" iyy="${r_arm_link_04_iyy}" iyz="${r_arm_link_04_iyz}" izz="${r_arm_link_04_izz}"
-		col_rpy="1.57 0 0" col_xyz="0.0219475 -0.008888 -0.1347982"
-		vis_rpy="0 0 0" vis_xyz="-0.00245 0.00175 -0.158"
-		radius="0.05"
-		length="${r_arm_link_04_length}"
-		mesh_file="package://dualarm_description/meshes/dualarm/r_arm4.STL"
-		mesh_scale="0.001 0.001 0.001"
-/>
-<m_joint_100
-		name="dualarm_joint6"
-		type="revolute"
-		axis_xyz="0 0 1"
-		origin_rpy="0 0 0"
-		origin_xyz="0 0 -0.242"
-		parent="${r_arm_link_03_name}"
-		child="${r_arm_link_04_name}"
-		limit_e="100" limit_l="-1.5708" limit_u="1.5708" limit_v="0"
-/>
-<m_link_cylinder
-		name="${r_arm_link_05_name}"
-		mass="${r_arm_link_05_mass}"
-		origin_rpy="0 0 0"
-		origin_xyz="0.0282566 -0.0026831 -0.1626786"
-		ixx="${r_arm_link_05_ixx}" ixy="${r_arm_link_05_ixy}" ixz="${r_arm_link_05_ixz}" iyy="${r_arm_link_05_iyy}" iyz="${r_arm_link_05_iyz}" izz="${r_arm_link_05_izz}"
-		col_rpy="0 0 0" col_xyz="0.0282566 -0.0026831 -0.1626786"
-		vis_rpy="0 0 0" vis_xyz="0 0 0"
-		radius="0.05"
-		length="${r_arm_link_05_length}"
-		mesh_file="package://dualarm_description/meshes/dualarm/r_arm5.STL"
-		mesh_scale="0.001 0.001 0.001"
-/>
-<m_joint_100
-		name="dualarm_joint7"
-		type="revolute"
-		axis_xyz="0 1 0"
-		origin_rpy="0 0 0"
-		origin_xyz="-0.0245 0.00175 -0.158"
-		parent="${r_arm_link_04_name}"
-		child="${r_arm_link_05_name}"
-		limit_e="100" limit_l="0" limit_u="2.3562" limit_v="1"
-/>
-<m_link_cylinder
-		name="${r_arm_link_06_name}"
-		mass="${r_arm_link_06_mass}"
-		origin_rpy="0 0 0"
-		origin_xyz="0 -0.0027174 -0.0051051"
-		ixx="${r_arm_link_06_ixx}" ixy="${r_arm_link_06_ixy}" ixz="${r_arm_link_06_ixz}" iyy="${r_arm_link_06_iyy}" iyz="${r_arm_link_06_iyz}" izz="${r_arm_link_06_izz}"
-		col_rpy="0 0 0" col_xyz="0 -0.0027174 -0.0051051"
-		vis_rpy="3.14 0 0" vis_xyz="-0.032 0.034 0.085"
-		radius="0.05"
-		length="${r_arm_link_06_length}"
-		mesh_file="package://dualarm_description/meshes/dualarm/link6.STL"
-		mesh_scale="0.001 0.001 0.001"
-/>
-<m_joint_100
-		name="dualarm_joint8"
-		type="revolute"
-		axis_xyz="0 0 1"
-		origin_rpy="0 0 0"
-		origin_xyz="0.0245 -0.00175 -0.235"
-		parent="${r_arm_link_05_name}"
-		child="${r_arm_link_06_name}"
-		limit_e="100" limit_l="-1.5708" limit_u="1.5708" limit_v="1"
-/>
-<!-- left_arm part-->
-<m_link_cylinder
-		name="${l_arm_link_01_name}"
-		mass="${l_arm_link_01_mass}"
-		origin_rpy="0 0 0"
-		origin_xyz="0.0002952 -0.0341703 0.076461"
-		ixx="${l_arm_link_01_ixx}"
-		ixy="${l_arm_link_01_ixy}"
-		ixz="${l_arm_link_01_ixz}" iyy="${l_arm_link_01_iyy}" iyz="${l_arm_link_01_iyz}" izz="${l_arm_link_01_izz}"
-		col_rpy="1.57 0 0" col_xyz="0.0002952 -0.0341703 0.076461"
-		vis_rpy="0 0 0" vis_xyz="0 -0.075 0.083"
-		radius="0.04"
-		length="${l_arm_link_01_length}"
-		mesh_file="package://dualarm_description/meshes/dualarm/l_arm1.STL"
-		mesh_scale="0.001 0.001 0.001"
-/>
-<m_joint_100
-		name="dualarm_joint9"
-		type="revolute"
-		axis_xyz="0 0 -1"
-		origin_rpy="0 0 0"
-		origin_xyz="0 -0.125 0.217"
-		parent="${waist_link_02_name}"
-		child="${l_arm_link_01_name}"
-		limit_e="100" limit_l="-1.5708" limit_u="0.5236" limit_v="1"
-/>
-<m_link_cylinder
-		name="${l_arm_link_02_name}"
-		mass="${l_arm_link_02_mass}"
-		origin_rpy="0 0 0"
-		origin_xyz="0.0112502 -0.0950175 0"
-		ixx="${l_arm_link_02_ixx}" ixy="${l_arm_link_02_ixy}" ixz="${l_arm_link_02_ixz}" iyy="${l_arm_link_02_iyy}" iyz="${l_arm_link_02_iyz}" izz="${l_arm_link_02_izz}"
-		col_rpy="0 -1.57 0" col_xyz="0.0112502 -0.0950175 0"
-		vis_rpy="0 0 0" vis_xyz="0 -0.11 -0.00"
-		radius="0.04"
-		length="${l_arm_link_02_length}"
-		mesh_file="package://dualarm_description/meshes/dualarm/l_arm2.STL"
-		mesh_scale="0.001 0.001 0.001"
-/>
-<m_joint_100
-		name="dualarm_joint10"
-		type="revolute"
-		axis_xyz="0 -1 0"
-		origin_rpy="0 0 0"
-		origin_xyz="0 -0.09 0.083"
-		parent="${l_arm_link_01_name}"
-		child="${l_arm_link_02_name}"
-		limit_e="100" limit_l="-1.5708" limit_u="0.7854" limit_v="1"
-/>
-<m_link_cylinder
-		name="${l_arm_link_03_name}"
-		mass="${l_arm_link_03_mass}"
-		origin_rpy="0 0 0"
-		origin_xyz="0.0015675 -0.0003615 -0.1633768"
-		ixx="${l_arm_link_03_ixx}" ixy="${l_arm_link_03_ixy}" ixz="${l_arm_link_03_ixz}" iyy="${l_arm_link_03_iyy}" iyz="${l_arm_link_03_iyz}" izz="${l_arm_link_03_izz}"
-		col_rpy="0 0 0" col_xyz="0.0015675 -0.0003615 -0.1633768"
-		vis_rpy="0 0 0" vis_xyz="0 0 -0.242"
-		radius="0.05"
-		length="${l_arm_link_03_length}"
-		mesh_file="package://dualarm_description/meshes/dualarm/l_arm3.STL"
-		mesh_scale="0.001 0.001 0.001"
-/>
-<m_joint_100
-		name="dualarm_joint11"
-		type="revolute"
-		axis_xyz="1 0 0"
-		origin_rpy="0 0 0"
-		origin_xyz="0 -0.11 0"
-		parent="${l_arm_link_02_name}"
-		child="${l_arm_link_03_name}"
-		limit_e="100" limit_l="-1.5708" limit_u="0.3490" limit_v="1"
-/>
-<m_link_cylinder
-		name="${l_arm_link_04_name}"
-		mass="${l_arm_link_04_mass}"
-		origin_rpy="0 0 0"
-		origin_xyz="0.0219475 0.008888 -0.1347982"
-		ixx="${l_arm_link_04_ixx}" ixy="${l_arm_link_04_ixy}" ixz="${l_arm_link_04_ixz}" iyy="${l_arm_link_04_iyy}" iyz="${l_arm_link_04_iyz}" izz="${l_arm_link_04_izz}"
-		col_rpy="-1.57 0 0" col_xyz="0.0219475 0.008888 -0.1347982"
-		vis_rpy="0 0 0" vis_xyz="-0.0245 -0.00175 -0.158"
-		radius="0.05"
-		length="${l_arm_link_04_length}"
-		mesh_file="package://dualarm_description/meshes/dualarm/l_arm4.STL"
-		mesh_scale="0.001 0.001 0.001"
-/>
-<m_joint_100
-		name="dualarm_joint12"
-		type="revolute"
-		axis_xyz="0 0 1"
-		origin_rpy="0 0 0"
-		origin_xyz="0 0 -0.242"
-		parent="${l_arm_link_03_name}"
-		child="${l_arm_link_04_name}"
-		limit_e="100" limit_l="-1.5708" limit_u="1.5708" limit_v="1"
-/>
-<m_link_cylinder
-		name="${l_arm_link_05_name}"
-		mass="${l_arm_link_05_mass}"
-		origin_rpy="0 0 0"
-		origin_xyz="0.0282566 0.0026831 -0.1626786"
-		ixx="${l_arm_link_05_ixx}" ixy="${l_arm_link_05_ixy}" ixz="${l_arm_link_05_ixz}" iyy="${l_arm_link_05_iyy}" iyz="${l_arm_link_05_iyz}" izz="${l_arm_link_05_izz}"
-		col_rpy="0 0 0" col_xyz="0.0282566 0.0026831 -0.1626786"
-		vis_rpy="0 0 0" vis_xyz="0 0 0"
-		radius="0.05"
-		length="0.158"
-		mesh_file="package://dualarm_description/meshes/dualarm/l_arm5.STL"
-		mesh_scale="0.001 0.001 0.001"
-/>
-<m_joint_100
-		name="dualarm_joint13"
-		type="revolute"
-		axis_xyz="0 -1 0"
-		origin_rpy="0 0 0"
-		origin_xyz="-0.0245 -0.00175 -0.158"
-		parent="${l_arm_link_04_name}"
-		child="${l_arm_link_05_name}"
-		limit_e="100" limit_l="0" limit_u="2.3562" limit_v="1"
-/>
-<m_link_cylinder
-		name="${l_arm_link_06_name}"
-		mass="${l_arm_link_06_mass}"
-		origin_rpy="0 0 0"
-		origin_xyz="0 0.0027174 -0.0051051"
-		ixx="${l_arm_link_06_ixx}" ixy="${l_arm_link_06_ixy}" ixz="${l_arm_link_06_ixz}" iyy="${l_arm_link_06_iyy}" iyz="${l_arm_link_06_iyz}" izz="${l_arm_link_06_izz}"
-		col_rpy="0 0 0" col_xyz="0 0.0027174 -0.0051051"
-		vis_rpy="3.14 0 0" vis_xyz="-0.032 0.034 0.085"
-		radius="0.05"
-		length="${l_arm_link_06_length}"
-		mesh_file="package://dualarm_description/meshes/dualarm/link6.STL"
-		mesh_scale="0.001 0.001 0.001"
-/>
-<m_joint_100
-		name="dualarm_joint14"
-		type="revolute"
-		axis_xyz="0 0 1"
-		origin_rpy="0 0 0"
-		origin_xyz="0.0245 0.00175 -0.235"
-		parent="${l_arm_link_05_name}"
-		child="${l_arm_link_06_name}"
-		limit_e="100" limit_l="-0.7854" limit_u="0.7854" limit_v="1"
-/>
+	<!-- Base parts -->
+	<link name = "world"/>
+	<joint name="base_joint" type="fixed">
+		<origin
+				xyz="0 0 0"
+				rpy="0 0 0"/>
+		<parent
+				link="world"/>
+		<child
+				link="dual_arm_base_link"/>
+	</joint>
+	<link name="dual_arm_base_link"/>
+	<joint name="dual_arm_base_joint" type="fixed">
+		<origin
+				xyz="0 0 0"
+				rpy="0 0 0"/>
+		<parent
+			link="dual_arm_base_link"/>
+		<child
+			link="${base_link_name}"/>
+	</joint>
+	<m_link_cylinder
+			name="${base_link_name}"
+			mass="${base_link_mass}"
+			origin_rpy= "0 0 0"
+			origin_xyz="0 0 0"
+			ixx="${base_link_ixx}"
+			ixy="${base_link_ixy}"
+			ixz="${base_link_ixz}"
+			iyy="${base_link_iyy}"
+			iyz="${base_link_iyz}"
+			izz="${base_link_izz}"
+			vis_rpy="0 0 ${M_PI}"
+			vis_xyz="0 0 0"
+			mesh_file="package://dualarm_description/meshes/dualarm/base.STL"
+			mesh_scale="0.001 0.001 0.001"
+	/>
+	<!-- waist part -->
+	<m_joint_100
+			name="dualarm_joint1"
+			type="revolute"
+			axis_xyz="0 0 1"
+			origin_rpy="0 0 0"
+			origin_xyz="0 0 0.352"
+			parent="${base_link_name}"
+			child="${waist_link_01_name}"
+			limit_effort="800"
+			limit_lower="-${M_PI/2}"
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