Commit message: CLIK update
update check

File: DualArm/dualarm_description/urdf/link_to_joint.xacro (robot description, xacro)
@@ -1,41 +1,69 @@
 <?xml version="1.0" ?>
 <robot xmlns:xacro="http://www.ros.org/wiki/xacro">
-  <xacro:macro name="m_joint_100" params="name type axis_xyz origin_rpy origin_xyz parent child limit_e limit_l limit_u limit_v">
+  <xacro:macro name="m_joint_100" params="name type axis_xyz origin_rpy origin_xyz parent child limit_effort limit_lower limit_upper limit_v">
     <joint name="${name}" type="${type}">
       <axis xyz="${axis_xyz}" />
-      <limit effort="${limit_e}" lower="${limit_l}" upper="${limit_u}" velocity="${limit_v}" />
-      <origin rpy="${origin_rpy}" xyz="${origin_xyz}" />
-      <parent link="${parent}" />
-      <child link="${child}" />
+      <limit
+              effort="${limit_effort}"
+              lower="${limit_lower}"
+              upper="${limit_upper}"
+              velocity="${limit_v}" />
+      <origin
+              rpy="${origin_rpy}"
+              xyz="${origin_xyz}" />
+      <parent
+              link="${parent}" />
+      <child
+              link="${child}" />
+      <dynamics damping="0.1" friction="0.1"/>
     </joint>
-    <transmission name="trans_${name}">
+    <transmission
+            name="trans_${name}">
       <type>transmission_interface/SimpleTransmission</type>
-      <joint name="${name}">
+      <joint
+              name="${name}">
         <hardwareInterface>hardware_interface/EffortJointInterface</hardwareInterface>
       </joint>
-      <actuator name="motor_${name}">
+      <actuator
+              name="motor_${name}">
         <hardwareInterface>hardware_interface/EffortJointInterface</hardwareInterface>
-        <mechanicalReduction>101</mechanicalReduction>
+        <mechanicalReduction>1</mechanicalReduction>
       </actuator>
     </transmission>
   </xacro:macro>
   <xacro:macro name="m_link_cylinder"
-               params="name origin_xyz origin_rpy col_xyz col_rpy vis_rpy vis_xyz radius length mass ixx ixy ixz iyy iyz izz mesh_file mesh_scale">
+               params="name origin_xyz origin_rpy vis_rpy vis_xyz mass ixx ixy ixz iyy iyz izz mesh_file mesh_scale">
     <link name="${name}">
       <inertial>
         <mass value="${mass}" />
-        <origin rpy="${origin_rpy}" xyz="${origin_xyz}" />
-        <inertia ixx="${ixx}" ixy="${ixy}" ixz="${ixz}" iyy="${iyy}" iyz="${iyz}" izz="${izz}" />
+        <origin
+                rpy="${origin_rpy}"
+                xyz="${origin_xyz}" />
+        <inertia
+                ixx="${ixx}"
+                ixy="${ixy}"
+                ixz="${ixz}"
+                iyy="${iyy}"
+                iyz="${iyz}"
+                izz="${izz}" />
       </inertial>
-      <collision>
-        <origin rpy="${col_rpy}" xyz="${col_xyz}" />
+      <!--<collision>
+        <origin
+                rpy="${vis_rpy}"
+                xyz="${vis_xyz}" />
         <geometry>
-          <cylinder radius="${radius}" length="${length}" />
+          <mesh
+                  filename="${mesh_file}"
+                  scale="${mesh_scale}"/>
         </geometry>
-      </collision>
+      </collision>-->
       <visual>
-        <origin rpy="${vis_rpy}" xyz="${vis_xyz}" />
+        <origin
+                rpy="${vis_rpy}"
+                xyz="${vis_xyz}" />
         <geometry>
-          <mesh filename="${mesh_file}" scale="${mesh_scale}"/>
+          <mesh
+                  filename="${mesh_file}"
+                  scale="${mesh_scale}"/>
         </geometry>
       </visual>
@@ -45,43 +73,36 @@
     <link name="${name}">
       <inertial>
-        <mass value="${mass}" />
-        <origin rpy="${origin_rpy}" xyz="${origin_xyz}" />
-        <inertia ixx="${ixx}" ixy="${ixy}" ixz="${ixz}" iyy="${iyy}" iyz="${iyz}" izz="${izz}" />
+        <mass
+                value="${mass}" />
+        <origin
+                rpy="${origin_rpy}"
+                xyz="${origin_xyz}" />
+        <inertia
+                ixx="${ixx}"
+                ixy="${ixy}"
+                ixz="${ixz}"
+                iyy="${iyy}"
+                iyz="${iyz}"
+                izz="${izz}" />
       </inertial>
       <collision>
-        <origin rpy="${origin_rpy}" xyz="${origin_xyz}" />
+        <origin
+                rpy="${origin_rpy}"
+                xyz="${origin_xyz}" />
         <geometry>
-          <box size="${size}" />
+          <box
+                  size="${size}" />
         </geometry>
       </collision>
       <visual>
-        <origin rpy="${origin_rpy}" xyz="${origin_xyz}" />
+        <origin
+                rpy="${origin_rpy}"
+                xyz="${origin_xyz}" />
         <geometry>
-          <box size="${size}" />
+          <box
+                  size="${size}" />
         </geometry>
       </visual>
     </link>
   </xacro:macro>
-  <xacro:macro name="m_link_mesh" params="name origin_xyz origin_rpy colvis_rpy colvis_xyz meshfile meshscale mass ixx ixy ixz iyy iyz izz">
-    <link name="${name}">
-      <inertial>
-        <mass value="${mass}" />
-        <origin rpy="${origin_rpy}" xyz="${origin_xyz}" />
-        <inertia ixx="${ixx}" ixy="${ixy}" ixz="${ixz}" iyy="${iyy}" iyz="${iyz}" izz="${izz}" />
-      </inertial>
-      <collision>
-        <origin rpy="${colvis_rpy}" xyz="${colvis_xyz}" />
-        <geometry>
-          <mesh filename="${meshfile}" scale="${meshscale}"/>
-        </geometry>
-      </collision>
-      <visual>
-        <origin rpy="${colvis_rpy}" xyz="${colvis_xyz}" />
-        <geometry>
-          <mesh filename="${meshfile}" scale="${meshscale}"/>
-        </geometry>
-        <material name="light_black"/>
-      </visual>
-    </link>
-  </xacro:macro>
 </robot>

File: DualArm/dualarm_description/urdf/robot_parameter.xacro (robot description, xacro)
@@ -1,5 +1,5 @@
 <?xml version="1.0" ?>
 <robot xmlns:xacro="http://www.ros.org/wiki/xacro">
-  <xacro:property name="m_pi" value="3.14159"/>
+  <xacro:property name="M_PI" value="3.14159"/>
 <!--base-->
   <xacro:property name="base_link_name" value="base_link" />
@@ -30,5 +30,5 @@
   <xacro:property name="r_arm_link_04_mass" value="2.49"/>
   <xacro:property name="r_arm_link_05_mass" value="1.86"/>
-  <xacro:property name="r_arm_link_06_mass" value="2.676"/>
+  <xacro:property name="r_arm_link_06_mass" value="0.0646"/>
   <xacro:property name="l_arm_link_01_mass" value="3.35"/>
   <xacro:property name="l_arm_link_02_mass" value="3.51"/>
@@ -37,20 +37,4 @@
   <xacro:property name="l_arm_link_05_mass" value="1.86"/>
   <xacro:property name="l_arm_link_06_mass" value="0.0646"/>
-<!-- link_length -->
-  <xacro:property name="base_link_length" value ="0.352"/>
-  <xacro:property name="waist_link_01_length" value ="0.148"/>
-  <xacro:property name="waist_link_02_length" value ="0.217"/>
-  <xacro:property name="r_arm_link_01_length" value ="0.083"/>
-  <xacro:property name="r_arm_link_02_length" value ="0.09"/>
-  <xacro:property name="r_arm_link_03_length" value ="0.242"/>
-  <xacro:property name="r_arm_link_04_length" value ="0.158"/>
-  <xacro:property name="r_arm_link_05_length" value ="0.235"/>
-  <xacro:property name="r_arm_link_06_length" value ="0.01"/>
-  <xacro:property name="l_arm_link_01_length" value ="0.083"/>
-  <xacro:property name="l_arm_link_02_length" value ="0.09"/>
-  <xacro:property name="l_arm_link_03_length" value ="0.242"/>
-  <xacro:property name="l_arm_link_04_length" value ="0.158"/>
-  <xacro:property name="l_arm_link_05_length" value ="0.235"/>
-  <xacro:property name="l_arm_link_06_length" value ="0.01"/>
 <!-- link_inertia -->
   <xacro:property name="base_link_ixx" value="0.0"/>
@@ -60,10 +44,10 @@
   <xacro:property name="base_link_izz" value="0.0"/>
   <xacro:property name="base_link_iyz" value="0.0"/>
-  <xacro:property name="waist_link_01_ixx" value="83854563.43e-9"/>
-  <xacro:property name="waist_link_01_ixy" value="-135841.54e-9"/>
-  <xacro:property name="waist_link_01_ixz" value="-625787.35e-9"/>
-  <xacro:property name="waist_link_01_iyy" value="70969371.34e-9"/>
-  <xacro:property name="waist_link_01_iyz" value="-15432807.98e-9"/>
-  <xacro:property name="waist_link_01_izz" value="53062013.96e-9"/>
+  <xacro:property name="waist_link_01_ixx" value="83854563.43E-9"/>
+  <xacro:property name="waist_link_01_ixy" value="-135841.54E-9"/>
+  <xacro:property name="waist_link_01_ixz" value="-625787.35E-9"/>
+  <xacro:property name="waist_link_01_iyy" value="70969371.34E-9"/>
+  <xacro:property name="waist_link_01_iyz" value="-15432807.98E-9"/>
+  <xacro:property name="waist_link_01_izz" value="53062013.96E-9"/>
   <xacro:property name="waist_link_02_ixx" value="0.1408"/>
   <xacro:property name="waist_link_02_ixy" value="0.0"/>
@@ -72,34 +56,34 @@
   <xacro:property name="waist_link_02_iyz" value="0.003643"/>
   <xacro:property name="waist_link_02_izz" value="0.1080"/>
-  <xacro:property name="r_arm_link_01_ixx" value="9155194.92e-9"/>
-  <xacro:property name="r_arm_link_01_ixy" value="163898.7e-9"/>
-  <xacro:property name="r_arm_link_01_ixz" value="-52182.13e-9"/>
-  <xacro:property name="r_arm_link_01_iyy" value="7656654.39e-9"/>
-  <xacro:property name="r_arm_link_01_iyz" value="-981692.47e-9"/>
-  <xacro:property name="r_arm_link_01_izz" value="6023745.1e-9"/>
-  <xacro:property name="r_arm_link_02_ixx" value="11833182.94e-9"/>
-  <xacro:property name="r_arm_link_02_ixy" value="245028.38e-9"/>
-  <xacro:property name="r_arm_link_02_ixz" value="-121068.48e-9"/>
-  <xacro:property name="r_arm_link_02_iyy" value="5963801.91e-9"/>
-  <xacro:property name="r_arm_link_02_iyz" value="-81204.78e-9"/>
-  <xacro:property name="r_arm_link_02_izz" value="12674379.1e-9"/>
-  <xacro:property name="r_arm_link_03_ixx" value="14349158.07e-9"/>
+  <xacro:property name="r_arm_link_01_ixx" value="9155194.92E-9"/>
+  <xacro:property name="r_arm_link_01_ixy" value="163898.7E-9"/>
+  <xacro:property name="r_arm_link_01_ixz" value="-52182.13E-9"/>
+  <xacro:property name="r_arm_link_01_iyy" value="7656654.39E-9"/>
+  <xacro:property name="r_arm_link_01_iyz" value="-981692.47E-9"/>
+  <xacro:property name="r_arm_link_01_izz" value="6023745.1E-9"/>
+  <xacro:property name="r_arm_link_02_ixx" value="11833182.94E-9"/>
+  <xacro:property name="r_arm_link_02_ixy" value="245028.38E-9"/>
+  <xacro:property name="r_arm_link_02_ixz" value="-121068.48E-9"/>
+  <xacro:property name="r_arm_link_02_iyy" value="5963801.91E-9"/>
+  <xacro:property name="r_arm_link_02_iyz" value="-81204.78E-9"/>
+  <xacro:property name="r_arm_link_02_izz" value="12674379.1E-9"/>
+  <xacro:property name="r_arm_link_03_ixx" value="14349158.07E-9"/>
   <xacro:property name="r_arm_link_03_ixy" value="0.0"/>
   <xacro:property name="r_arm_link_03_ixz" value="0.0"/>
-  <xacro:property name="r_arm_link_03_iyy" value="15957517.14e-9"/>
-  <xacro:property name="r_arm_link_03_iyz" value="-1126404.95e-9"/>
-  <xacro:property name="r_arm_link_03_izz" value="3811118.16e-9"/>
-  <xacro:property name="r_arm_link_04_ixx" value="12305788.09e-9"/>
+  <xacro:property name="r_arm_link_03_iyy" value="15957517.14E-9"/>
+  <xacro:property name="r_arm_link_03_iyz" value="-1126404.95E-9"/>
+  <xacro:property name="r_arm_link_03_izz" value="3811118.16E-9"/>
+  <xacro:property name="r_arm_link_04_ixx" value="12305788.09E-9"/>
   <xacro:property name="r_arm_link_04_ixy" value="0.0"/>
-  <xacro:property name="r_arm_link_04_ixz" value="1326295.35e-9"/>
-  <xacro:property name="r_arm_link_04_iyy" value="10949889.37e-9"/>
-  <xacro:property name="r_arm_link_04_iyz" value="-322614.65e-9"/>
-  <xacro:property name="r_arm_link_04_izz" value="3675298.10e-9"/>
-  <xacro:property name="r_arm_link_05_ixx" value="4927170.75e-9"/>
+  <xacro:property name="r_arm_link_04_ixz" value="1326295.35E-9"/>
+  <xacro:property name="r_arm_link_04_iyy" value="10949889.37E-9"/>
+  <xacro:property name="r_arm_link_04_iyz" value="-322614.65E-9"/>
+  <xacro:property name="r_arm_link_04_izz" value="3675298.10E-9"/>
+  <xacro:property name="r_arm_link_05_ixx" value="4927170.75E-9"/>
   <xacro:property name="r_arm_link_05_ixy" value="0.0"/>
-  <xacro:property name="r_arm_link_05_ixz" value="-353301.92e-9"/>
-  <xacro:property name="r_arm_link_05_iyy" value="4076854.09e-9"/>
-  <xacro:property name="r_arm_link_05_iyz" value="298769.64e-9"/>
-  <xacro:property name="r_arm_link_05_izz" value="2250292.68e-9"/>
+  <xacro:property name="r_arm_link_05_ixz" value="-353301.92E-9"/>
+  <xacro:property name="r_arm_link_05_iyy" value="4076854.09E-9"/>
+  <xacro:property name="r_arm_link_05_iyz" value="298769.64E-9"/>
+  <xacro:property name="r_arm_link_05_izz" value="2250292.68E-9"/>
   <xacro:property name="r_arm_link_06_ixx" value="0.00005"/>
   <xacro:property name="r_arm_link_06_ixy" value="0.0"/>
@@ -114,28 +98,28 @@
   <xacro:property name="l_arm_link_01_iyz" value="-0.0005"/>
   <xacro:property name="l_arm_link_01_izz" value="0.0044"/>
-  <xacro:property name="l_arm_link_02_ixx" value="11625561.71e-9"/>
-  <xacro:property name="l_arm_link_02_ixy" value="-73542.31e-9"/>
-  <xacro:property name="l_arm_link_02_ixz" value="2404534.61e-9"/>
-  <xacro:property name="l_arm_link_02_iyy" value="6340663.94e-9"/>
-  <xacro:property name="l_arm_link_02_iyz" value="817088484.13e-9"/>
-  <xacro:property name="l_arm_link_02_izz" value="13098282.6e-9"/>
-  <xacro:property name="l_arm_link_03_ixx" value="14349157.75e-9"/>
+  <xacro:property name="l_arm_link_02_ixx" value="11625561.71E-9"/>
+  <xacro:property name="l_arm_link_02_ixy" value="-73542.31E-9"/>
+  <xacro:property name="l_arm_link_02_ixz" value="2404534.61E-9"/>
+  <xacro:property name="l_arm_link_02_iyy" value="6340663.94E-9"/>
+  <xacro:property name="l_arm_link_02_iyz" value="817088484.13E-9"/>
+  <xacro:property name="l_arm_link_02_izz" value="13098282.6E-9"/>
+  <xacro:property name="l_arm_link_03_ixx" value="14349157.75E-9"/>
   <xacro:property name="l_arm_link_03_ixy" value="0.0"/>
-  <xacro:property name="l_arm_link_03_ixz" value="-1118640.19e-9"/>
-  <xacro:property name="l_arm_link_03_iyy" value="15959292.97e-9"/>
+  <xacro:property name="l_arm_link_03_ixz" value="-1118640.19E-9"/>
+  <xacro:property name="l_arm_link_03_iyy" value="15959292.97E-9"/>
   <xacro:property name="l_arm_link_03_iyz" value="0.0007"/>
-  <xacro:property name="l_arm_link_03_izz" value="3812893.68e-9"/>
-  <xacro:property name="l_arm_link_04_ixx" value="12366056.79e-9"/>
+  <xacro:property name="l_arm_link_03_izz" value="3812893.68E-9"/>
+  <xacro:property name="l_arm_link_04_ixx" value="12366056.79E-9"/>
   <xacro:property name="l_arm_link_04_ixy" value="0.0"/>
-  <xacro:property name="l_arm_link_04_ixz" value="1314062.31e-9"/>
-  <xacro:property name="l_arm_link_04_iyy" value="11004463.34e-9"/>
+  <xacro:property name="l_arm_link_04_ixz" value="1314062.31E-9"/>
+  <xacro:property name="l_arm_link_04_iyy" value="11004463.34E-9"/>
   <xacro:property name="l_arm_link_04_iyz" value="0.0"/>
-  <xacro:property name="l_arm_link_04_izz" value="3670383.10e-9"/>
-  <xacro:property name="l_arm_link_05_ixx" value="4932126.5e-9"/>
-  <xacro:property name="l_arm_link_05_ixy" value="80829.44e-9"/>
-  <xacro:property name="l_arm_link_05_ixz" value="-353301.92e-9"/>
-  <xacro:property name="l_arm_link_05_iyy" value="4076854.09e-9"/>
-  <xacro:property name="l_arm_link_05_iyz" value="-355897.62e-9"/>
-  <xacro:property name="l_arm_link_05_izz" value="2255248.43e-9"/>
+  <xacro:property name="l_arm_link_04_izz" value="3670383.10E-9"/>
+  <xacro:property name="l_arm_link_05_ixx" value="4932126.5E-9"/>
+  <xacro:property name="l_arm_link_05_ixy" value="80829.44E-9"/>
+  <xacro:property name="l_arm_link_05_ixz" value="-353301.92E-9"/>
+  <xacro:property name="l_arm_link_05_iyy" value="4076854.09E-9"/>
+  <xacro:property name="l_arm_link_05_iyz" value="-355897.62E-9"/>
+  <xacro:property name="l_arm_link_05_izz" value="2255248.43E-9"/>
   <xacro:property name="l_arm_link_06_ixx" value="0.00005"/>
   <xacro:property name="l_arm_link_06_ixy" value="0.0"/>
@@ -144,4 +128,3 @@
   <xacro:property name="l_arm_link_06_iyz" value="0.0"/>
   <xacro:property name="l_arm_link_06_izz" value="0.00005"/>
-  <xacro:property name="l_arm_link_06_z" value="170.1051"/>
 </robot>
