Commit message: #3 fix xacro model
fix the dualarm parameters & stl files

File: DualArm/dualarm_description/urdf/dual_arm.urdf (robot description, URDF)
Before this commit: robot dualarm, 21 links, 20 joints
Links:
- link link_01: mass 11.91 -> 6.61; geometry visual mesh filename=package://dualarm_description/meshes/stl/waist1.STL scale=0.001 0.001 0.001
- link link_02: mass 9.901 -> 8.2662; geometry visual mesh filename=package://dualarm_description/meshes/stl/waist2.STL scale=0.001 0.001 0.001
- link link_03: mass 3.35 -> 2.8163; geometry visual mesh filename=package://dualarm_description/meshes/stl/r1.STL scale=0.001 0.001 0.001
- link link_04: mass 3.51 -> 3.213; geometry visual mesh filename=package://dualarm_description/meshes/stl/r2.STL scale=0.001 0.001 0.001
- link link_05: mass 2.59 -> 2.4856; geometry visual mesh filename=package://dualarm_description/meshes/stl/r3.STL scale=0.001 0.001 0.001
- link link_06: mass 2.49 -> 2.1204; geometry visual mesh filename=package://dualarm_description/meshes/stl/r4.STL scale=0.001 0.001 0.001
- link link_07: mass 1.86 -> 1.8777; geometry visual mesh filename=package://dualarm_description/meshes/stl/r5.STL scale=0.001 0.001 0.001
- link link_08: mass 2.676 -> 2.6999; geometry visual mesh filename=package://dualarm_description/meshes/stl/r6.STL scale=0.001 0.001 0.001
- link link_10: mass 3.35 -> 2.8163; geometry visual mesh filename=package://dualarm_description/meshes/stl/l1.STL scale=0.001 0.001 0.001
- link link_11: mass 3.51 -> 3.213; geometry visual mesh filename=package://dualarm_description/meshes/stl/l2.STL scale=0.001 0.001 0.001
- link link_12: mass 2.59 -> 2.4856; geometry visual mesh filename=package://dualarm_description/meshes/stl/l3.STL scale=0.001 0.001 0.001
- link link_13: mass 2.49 -> 2.1204; geometry visual mesh filename=package://dualarm_description/meshes/stl/l4.STL scale=0.001 0.001 0.001
- link link_14: mass 1.86 -> 1.8777; geometry visual mesh filename=package://dualarm_description/meshes/stl/l5.STL scale=0.001 0.001 0.001
- link link_15: mass 2.1946 -> 2.6999; geometry visual mesh filename=package://dualarm_description/meshes/stl/l6.STL scale=0.001 0.001 0.001
- link link_L_hand: mass 1.29 -> 1.5
- link link_R_hand: mass 1.29 -> 1.6338; geometry visual mesh filename=package://dualarm_description/meshes/stl/r7.STL scale=0.001 0.001 0.001
- link robot_base_link: geometry visual mesh filename=package://dualarm_description/meshes/stl/base.STL scale=0.001 0.001 0.001
Joints:
- joint dual_arm_base_joint: origin xyz=0 0 0 rpy=0 0 0 -> xyz=0 0 0.3 rpy=0 0 0
- joint dualarm_L_end: origin xyz=0 0 -0.122 rpy=0 0 0 -> xyz=0 0 -0.04681 rpy=0 0 0
- joint dualarm_R_end: origin xyz=0 0 -0.122 rpy=0 0 0 -> xyz=0 0 -0.04681 rpy=0 0 0
- joint dualarm_joint1: origin xyz=0 0 0.652 rpy=0 0 0 -> xyz=0 0 0.3031 rpy=0 0 0
- joint dualarm_joint10: origin xyz=0 0.125 0.217 rpy=0 0 0 -> xyz=0 0.125 0.18565 rpy=0 0 0
- joint dualarm_joint11: origin xyz=0 0.09 0.083 rpy=0 0 0 -> xyz=0 0.05265 0.11435 rpy=0 0 0
- joint dualarm_joint12: origin xyz=0 0.11 0 rpy=0 0 0 -> xyz=0 0.14735 0 rpy=0 0 0
- joint dualarm_joint13: origin xyz=0 0 -0.242 rpy=0 0 0 -> xyz=0 0 -0.21425 rpy=0 0 0
- joint dualarm_joint14: origin xyz=-0.0245 0 -0.158 rpy=0 0 0 -> xyz=-0.0245 0 -0.18575 rpy=0 0 0
- joint dualarm_joint15: origin xyz=0.0245 0 -0.155 rpy=0 0 0 -> xyz=0.0245 0 -0.14 rpy=0 0 0
- joint dualarm_joint16: origin xyz=0 0 -0.0755 rpy=0 0 0 -> xyz=0 0 -0.091 rpy=0 0 0
- joint dualarm_joint2: origin xyz=0 0 0.148 rpy=0 0 0 -> xyz=0 0 0.1969 rpy=0 0 0
- joint dualarm_joint3: origin xyz=0 -0.125 0.217 rpy=0 0 0 -> xyz=0 -0.125 0.18565 rpy=0 0 0
- joint dualarm_joint4: origin xyz=0 -0.09 0.083 rpy=0 0 0 -> xyz=0 -0.05265 0.11435 rpy=0 0 0
- joint dualarm_joint5: origin xyz=0 -0.11 0 rpy=0 0 0 -> xyz=0 -0.14735 0 rpy=0 0 0
- joint dualarm_joint6: origin xyz=0 0 -0.242 rpy=0 0 0 -> xyz=0 0 -0.21425 rpy=0 0 0
- joint dualarm_joint7: origin xyz=-0.0245 0 -0.158 rpy=0 0 0 -> xyz=-0.0245 0 -0.18575 rpy=0 0 0
- joint dualarm_joint8: origin xyz=0.0245 0 -0.155 rpy=0 0 0 -> xyz=0.0245 0 -0.14 rpy=0 0 0
- joint dualarm_joint9: origin xyz=0 0 -0.0755 rpy=0 0 0 -> xyz=0 0 -0.091 rpy=0 0 0

File: DualArm/dualarm_description/urdf/dual_arm.xacro (robot description, xacro)
@@ -18,5 +18,5 @@
 	<joint name="dual_arm_base_joint" type="fixed">
 		<origin
-			xyz="0 0 0"
+			xyz="0 0 0.3"
 			rpy="0 0 0"/>
 		<parent
@@ -30,5 +30,5 @@
 			<origin
 					rpy="0 0 0"
-					xyz="0 0 0" />
+					xyz="0 0 0.15" />
 			<inertia
 					ixx="${base_link_ixx}"
@@ -41,9 +41,9 @@
 		<visual>
 			<origin
-					rpy="0 0 ${M_PI}"
-					xyz="0 0 0.3" />
-			<geometry>
-				<mesh
-						filename="package://dualarm_description/meshes/dualarm/base.STL"
+					rpy="0 0 0"
+					xyz="0 0 0" />
+			<geometry>
+				<mesh
+						filename="package://dualarm_description/meshes/stl/base.STL"
 						scale="0.001 0.001 0.001"/>
 			</geometry>
@@ -60,5 +60,5 @@
 		<origin
 				rpy="0 0 0"
-				xyz="0 0 0.652" />
+				xyz="0 0 0.3031" />
 		<parent
 				link="${base_link_name}" />
@@ -85,5 +85,5 @@
 			<origin
 					rpy="0 0 0"
-					xyz="-0.0001 -0.00305 0.09799" />
+					xyz="-0.0001211 -0.0015722 0.1519998" />
 			<inertia
 					ixx="${waist_link_01_ixx}"
@@ -100,5 +100,5 @@
 			<geometry>
 				<mesh
-						filename="package://dualarm_description/meshes/dualarm1/link1.STL"
+						filename="package://dualarm_description/meshes/stl/waist1.STL"
 						scale="0.001 0.001 0.001"/>
 			</geometry>
@@ -114,5 +114,5 @@
 		<origin
 				rpy="0 0 0"
-				xyz="0 0 0.148" />
+				xyz="0 0 0.1969" />
 		<parent
 				link="${waist_link_01_name}" />
@@ -139,5 +139,5 @@
 			<origin
 					rpy="0 0 0"
-					xyz="0.0010139 0.0036731 0.1436171" />
+					xyz="0.00597 0.0059226 0.1235" />
 			<inertia
 					ixx="${waist_link_02_ixx}"
@@ -154,5 +154,5 @@
 			<geometry>
 				<mesh
-						filename="package://dualarm_description/meshes/dualarm/waist_2.STL"
+						filename="package://dualarm_description/meshes/stl/waist2.STL"
 						scale="0.001 0.001 0.001"/>
 			</geometry>
@@ -171,5 +171,5 @@
 		<origin
 				rpy="0 0 0"
-				xyz="0 -0.125 0.217" />
+				xyz="0 -0.125 0.18565" />
 		<parent
 				link="${waist_link_02_name}" />
@@ -196,5 +196,5 @@
 			<origin
 					rpy="0 0 0"
-					xyz="-0.0007 0.01789 0.06438" />
+					xyz="-0.0007018 -0.0179392 0.0955618" />
 			<inertia
 					ixx="${r_arm_link_01_ixx}"
@@ -211,5 +211,5 @@
 			<geometry>
 				<mesh
-						filename="package://dualarm_description/meshes/dualarm1/link3.STL"
+						filename="package://dualarm_description/meshes/stl/r1.STL"
 						scale="0.001 0.001 0.001"/>
 			</geometry>
@@ -225,5 +225,5 @@
 		<origin
 				rpy="0 0 0"
-				xyz="0 -0.09 0.083" />
+				xyz="0 -0.05265 0.11435" />
 		<parent
 				link="${r_arm_link_01_name}" />
@@ -250,5 +250,5 @@
 			<origin
 					rpy="0 0 0"
-					xyz="-0.00021 -0.07804 0.00077" />
+					xyz="-0.00021 -0.1153861 0.00077" />
 			<inertia
 					ixx="${r_arm_link_02_ixx}"
@@ -265,5 +265,5 @@
 			<geometry>
 				<mesh
-						filename="package://dualarm_description/meshes/dualarm1/link4.STL"
+						filename="package://dualarm_description/meshes/stl/r2.STL"
 						scale="0.001 0.001 0.001"/>
 			</geometry>
@@ -279,5 +279,5 @@
 		<origin
 				rpy="0 0 0"
-				xyz="0 -0.11 0" />
+				xyz="0 -0.14735 0" />
 		<parent
 				link="${r_arm_link_02_name}" />
@@ -304,5 +304,5 @@
 			<origin
 					rpy="0 0 0"
-					xyz="-0.00254 -0.00018 -0.15039" />
+					xyz="-0.0025431 -0.0001796 -0.1503879" />
 			<inertia
 					ixx="${r_arm_link_03_ixx}"
@@ -319,5 +319,5 @@
 			<geometry>
 				<mesh
-						filename="package://dualarm_description/meshes/dualarm1/link5.STL"
+						filename="package://dualarm_description/meshes/stl/r3.STL"
 						scale="0.001 0.001 0.001"/>
 			</geometry>
@@ -333,5 +333,5 @@
 		<origin
 				rpy="0 0 0"
-				xyz="0 0 -0.242" />
+				xyz="0 0 -0.21425" />
 		<parent
 				link="${r_arm_link_03_name}" />
@@ -358,5 +358,5 @@
 			<origin
 					rpy="0 0 0"
-					xyz="-0.01909 0.00259 -0.10869" />
+					xyz="-0.0191 0.0026 -0.1364" />
 			<inertia
 					ixx="${r_arm_link_04_ixx}"
@@ -373,5 +373,5 @@
 			<geometry>
 				<mesh
-						filename="package://dualarm_description/meshes/dualarm1/link6.STL"
+						filename="package://dualarm_description/meshes/stl/r4.STL"
 						scale="0.001 0.001 0.001"/>
 			</geometry>
@@ -387,5 +387,5 @@
 		<origin
 				rpy="0 0 0"
-				xyz="-0.0245 0 -0.158" />
+				xyz="-0.0245 0 -0.18575" />
 		<parent
 				link="${r_arm_link_04_name}" />
@@ -412,5 +412,5 @@
 			<origin
 					rpy="0 0 0"
-					xyz="0.02217 0.00213 -0.09649" />
+					xyz="-0.0023 0.0022 -0.0965" />
 			<inertia
 					ixx="${r_arm_link_05_ixx}"
@@ -427,5 +427,5 @@
 			<geometry>
 				<mesh
-						filename="package://dualarm_description/meshes/dualarm1/link7.STL"
+						filename="package://dualarm_description/meshes/stl/r5.STL"
 						scale="0.001 0.001 0.001"/>
 			</geometry>
@@ -441,5 +441,5 @@
 		<origin
 				rpy="0 0 0"
-				xyz="0.0245 0 -0.155" />
+				xyz="0.0245 0 -0.14" />
 		<parent
 				link="${r_arm_link_05_name}" />
@@ -466,5 +466,5 @@
 			<origin
 					rpy="0 0 0"
-					xyz="0.00173 -0.00014 -0.13722" />
+					xyz="0.0036 -0.0004 -0.0746" />
 			<inertia
 					ixx="${r_arm_link_06_ixx}"
@@ -481,5 +481,5 @@
 			<geometry>
 				<mesh
-						filename="package://dualarm_description/meshes/dualarm1/Wrist.STL"
+						filename="package://dualarm_description/meshes/stl/r6.STL"
 						scale="0.001 0.001 0.001"/>
 			</geometry>
@@ -495,5 +495,5 @@
 		<origin
 				rpy="0 0 0"
-				xyz="0 0 -0.0755" />
+				xyz="0 0 -0.091" />
 		<parent
 				link="${r_arm_link_06_name}" />
@@ -520,5 +520,5 @@
 			<origin
 					rpy="0 0 0"
-					xyz="0 0 0" />
+					xyz="0.0099 0.0087 -0.126" />
 			<inertia
 					ixx="${r_arm_link_07_ixx}"
@@ -535,5 +535,5 @@
 			<geometry>
 				<mesh
-						filename="package://dualarm_description/meshes/dualarm1/Allegro_wrist.STL"
+						filename="package://dualarm_description/meshes/stl/r7.STL"
 						scale="0.001 0.001 0.001"/>
 			</geometry>
@@ -541,5 +541,6 @@
 	</link>
 	<joint name="dualarm_R_end" type="fixed">
-		<origin xyz="0 0 -0.122"
+		<origin
+				xyz="0 0 -0.04681"
 				rpy="0 0 0"/>
 		<parent link="${r_arm_link_hand}"/>
@@ -557,5 +558,5 @@
 		<origin
 				rpy="0 0 0"
-				xyz="0 0.125 0.217" />
+				xyz="0 0.125 0.18565" />
 		<parent
 				link="${waist_link_02_name}" />
@@ -582,5 +583,5 @@
 			<origin
 					rpy="0 0 0"
-					xyz="-0.00087 0.017 0.064" />
+					xyz="-0.0009 0.0179 0.0957" />
 			<inertia
 					ixx="${l_arm_link_01_ixx}"
@@ -593,9 +594,9 @@
 		<visual>
 			<origin
-					rpy="0 0 ${M_PI}"
-					xyz="0 0 0" />
-			<geometry>
-				<mesh
-						filename="package://dualarm_description/meshes/dualarm1/link3.STL"
+					rpy="0 0 0"
+					xyz="0 0 0" />
+			<geometry>
+				<mesh
+						filename="package://dualarm_description/meshes/stl/l1.STL"
 						scale="0.001 0.001 0.001"/>
 			</geometry>
@@ -611,5 +612,5 @@
 		<origin
 				rpy="0 0 0"
-				xyz="0 0.09 0.083" />
+				xyz="0 0.05265 0.11435" />
 		<parent
 				link="${l_arm_link_01_name}" />
@@ -636,5 +637,5 @@
 			<origin
 					rpy="0 0 0"
-					xyz="0.00089 0.07577 0.00053" />
+					xyz="0.0009 0.1131 0.0005" />
 			<inertia
 					ixx="${l_arm_link_02_ixx}"
@@ -647,9 +648,9 @@
 		<visual>
 			<origin
-					rpy="${M_PI} 0 0"
-					xyz="0 -0.011 0" />
-			<geometry>
-				<mesh
-						filename="package://dualarm_description/meshes/dualarm1/link4.STL"
+					rpy="0 0 0"
+					xyz="0 0 0" />
+			<geometry>
+				<mesh
+						filename="package://dualarm_description/meshes/stl/l2.STL"
 						scale="0.001 0.001 0.001"/>
 			</geometry>
@@ -665,5 +666,5 @@
 		<origin
 				rpy="0 0 0"
-				xyz="0 0.11 0" />
+				xyz="0 0.14735 0" />
 		<parent
 				link="${l_arm_link_02_name}" />
@@ -690,5 +691,5 @@
 			<origin
 					rpy="0 0 0"
-					xyz="-0.00238 0.00016 -0.15039" />
+					xyz="-0.0024 0.0002 -0.1504" />
 			<inertia
 					ixx="${l_arm_link_03_ixx}"
@@ -705,5 +706,5 @@
 			<geometry>
 				<mesh
-						filename="package://dualarm_description/meshes/dualarm1/link5.STL"
+						filename="package://dualarm_description/meshes/stl/l3.STL"
 						scale="0.001 0.001 0.001"/>
 			</geometry>
@@ -719,5 +720,5 @@
 		<origin
 				rpy="0 0 0"
-				xyz="0 0 -0.242" />
+				xyz="0 0 -0.21425" />
 		<parent
 				link="${l_arm_link_03_name}" />
@@ -744,5 +745,5 @@
 			<origin
 					rpy="0 0 0"
-					xyz="-0.01891 -0.00275 -0.11422" />
+					xyz="-0.0189 -0.0027 -0.136" />
 			<inertia
 					ixx="${l_arm_link_04_ixx}"
@@ -759,5 +760,5 @@
 			<geometry>
 				<mesh
-						filename="package://dualarm_description/meshes/dualarm1/link6.STL"
+						filename="package://dualarm_description/meshes/stl/l4.STL"
 						scale="0.001 0.001 0.001"/>
 			</geometry>
@@ -773,5 +774,5 @@
 		<origin
 				rpy="0 0 0"
-				xyz="-0.0245 0 -0.158" />
+				xyz="-0.0245 0 -0.18575" />
 		<parent
 				link="${l_arm_link_04_name}" />
@@ -798,5 +799,5 @@
 			<origin
 					rpy="0 0 0"
-					xyz="0.02219 -0.00137 -0.09649" />
+					xyz="-0.0023 -0.0014 -0.0965" />
 			<inertia
 					ixx="${l_arm_link_05_ixx}"
@@ -813,5 +814,5 @@
 			<geometry>
 				<mesh
-						filename="package://dualarm_description/meshes/dualarm1/link7.STL"
+						filename="package://dualarm_description/meshes/stl/l5.STL"
 						scale="0.001 0.001 0.001"/>
 			</geometry>
@@ -827,5 +828,5 @@
 		<origin
 				rpy="0 0 0"
-				xyz="0.0245 0 -0.155" />
+				xyz="0.0245 0 -0.14" />
 		<parent
 				link="${l_arm_link_05_name}" />
@@ -852,5 +853,5 @@
 			<origin
 					rpy="0 0 0"
-					xyz="0.00173 0.00014 -0.13722" />
+					xyz="0.0039 -0.0002 -0.08" />
 			<inertia
 					ixx="${l_arm_link_06_ixx}"
@@ -867,5 +868,5 @@
 			<geometry>
 				<mesh
-						filename="package://dualarm_description/meshes/dualarm1/Wrist.STL"
+						filename="package://dualarm_description/meshes/stl/l6.STL"
 						scale="0.001 0.001 0.001"/>
 			</geometry>
@@ -881,5 +882,5 @@
 		<origin
 				rpy="0 0 0"
-				xyz="0 0 -0.0755" />
+				xyz="0 0 -0.091" />
 		<parent
 				link="${l_arm_link_06_name}" />
@@ -906,5 +907,5 @@
 			<origin
 					rpy="0 0 0"
-					xyz="0 0 0" />
+					xyz="0.0099 -0.0087 -0.126" />
 			<inertia
 					ixx="${l_arm_link_07_ixx}"
@@ -927,5 +928,6 @@
 	</link>
 	<joint name="dualarm_L_end" type="fixed">
-		<origin xyz="0 0 -0.122"
+		<origin
+				xyz="0 0 -0.04681"
 				rpy="0 0 0"/>
 		<parent link="${l_arm_link_hand}"/>
