Commit message: #3.1 fix xacro model
update param

File: DualArm/dualarm_description/urdf/dual_arm.urdf (robot description, URDF)
Before this commit: robot dualarm, 21 links, 20 joints
Links:
- link link_01: mass 6.61 -> 11.91
- link link_02: mass 8.2662 -> 10.901
- link link_03: mass 2.8163 -> 3.35
- link link_04: mass 3.213 -> 3.51
- link link_05: mass 2.4856 -> 2.59
- link link_06: mass 2.1204 -> 2.49
- link link_07: mass 1.8777 -> 1.8
- link link_08: mass 2.6999 -> 1.73
- link link_10: mass 2.8163 -> 3.35
- link link_11: mass 3.213 -> 3.51
- link link_12: mass 2.4856 -> 2.59
- link link_13: mass 2.1204 -> 2.49
- link link_14: mass 1.8777 -> 1.8
- link link_15: mass 2.6999 -> 1.73
- link link_L_hand: mass 1.5 -> 1.147; geometry visual mesh filename=package://dualarm_description/meshes/stl/hand_adapter_L.STL scale=0.001 0.001 0.001
- link link_R_hand: mass 1.6338 -> 1.08
Joints:
- joint dual_arm_base_joint: origin xyz=0 0 0.3 rpy=0 0 0 -> xyz=0 0 0 rpy=0 0 0

File: DualArm/dualarm_description/urdf/dual_arm.xacro (robot description, xacro)
@@ -18,5 +18,5 @@
 	<joint name="dual_arm_base_joint" type="fixed">
 		<origin
-			xyz="0 0 0.3"
+			xyz="0 0 0"
 			rpy="0 0 0"/>
 		<parent
@@ -139,5 +139,5 @@
 			<origin
 					rpy="0 0 0"
-					xyz="0.00597 0.0059226 0.1235" />
+					xyz="0.0054 0.0042 0.119" />
 			<inertia
 					ixx="${waist_link_02_ixx}"
@@ -907,5 +907,5 @@
 			<origin
 					rpy="0 0 0"
-					xyz="0.0099 -0.0087 -0.126" />
+					xyz="0.0188 -0.0157 -0.1202" />
 			<inertia
 					ixx="${l_arm_link_07_ixx}"
@@ -922,5 +922,5 @@
 			<geometry>
 				<mesh
-						filename="package://dualarm_description/meshes/dualarm1/hand_adapter_L.STL"
+						filename="package://dualarm_description/meshes/stl/hand_adapter_L.STL"
 						scale="0.001 0.001 0.001"/>
 			</geometry>

File: DualArm/dualarm_description/urdf/robot_parameter.xacro (robot description, xacro)
@@ -25,20 +25,20 @@
 <!-- link_mass -->
   <xacro:property name="base_link_mass" value="10.0"/>
-  <xacro:property name="waist_link_01_mass" value="6.61"/>
-  <xacro:property name="waist_link_02_mass" value="8.2662"/>
-  <xacro:property name="r_arm_link_01_mass" value="2.8163"/>
-  <xacro:property name="r_arm_link_02_mass" value="3.213"/>
-  <xacro:property name="r_arm_link_03_mass" value="2.4856"/>
-  <xacro:property name="r_arm_link_04_mass" value="2.1204"/>
-  <xacro:property name="r_arm_link_05_mass" value="1.8777"/>
-  <xacro:property name="r_arm_link_06_mass" value="2.6999"/>
-  <xacro:property name="r_arm_link_07_mass" value="1.6338"/>
-  <xacro:property name="l_arm_link_01_mass" value="2.8163"/>
-  <xacro:property name="l_arm_link_02_mass" value="3.213"/>
-  <xacro:property name="l_arm_link_03_mass" value="2.4856"/>
-  <xacro:property name="l_arm_link_04_mass" value="2.1204"/>
-  <xacro:property name="l_arm_link_05_mass" value="1.8777"/>
-  <xacro:property name="l_arm_link_06_mass" value="2.6999"/>
-  <xacro:property name="l_arm_link_07_mass" value="1.5"/>
+  <xacro:property name="waist_link_01_mass" value="11.91"/>
+  <xacro:property name="waist_link_02_mass" value="10.901"/>
+  <xacro:property name="r_arm_link_01_mass" value="3.35"/>
+  <xacro:property name="r_arm_link_02_mass" value="3.51"/>
+  <xacro:property name="r_arm_link_03_mass" value="2.59"/>
+  <xacro:property name="r_arm_link_04_mass" value="2.49"/>
+  <xacro:property name="r_arm_link_05_mass" value="1.8"/>
+  <xacro:property name="r_arm_link_06_mass" value="1.73"/>
+  <xacro:property name="r_arm_link_07_mass" value="1.08"/>
+  <xacro:property name="l_arm_link_01_mass" value="3.35"/>
+  <xacro:property name="l_arm_link_02_mass" value="3.51"/>
+  <xacro:property name="l_arm_link_03_mass" value="2.59"/>
+  <xacro:property name="l_arm_link_04_mass" value="2.49"/>
+  <xacro:property name="l_arm_link_05_mass" value="1.8"/>
+  <xacro:property name="l_arm_link_06_mass" value="1.73"/>
+  <xacro:property name="l_arm_link_07_mass" value="1.147"/>
 <!-- link_inertia -->
   <xacro:property name="base_link_ixx" value="0.0"/>
@@ -48,99 +48,99 @@
   <xacro:property name="base_link_izz" value="0.0"/>
   <xacro:property name="base_link_iyz" value="0.0"/>
-  <xacro:property name="waist_link_01_ixx" value="0.0522"/>
-  <xacro:property name="waist_link_01_ixy" value="-0.0001"/>
-  <xacro:property name="waist_link_01_ixz" value="0.0"/>
-  <xacro:property name="waist_link_01_iyy" value="0.0395"/>
-  <xacro:property name="waist_link_01_iyz" value="0.0003"/>
-  <xacro:property name="waist_link_01_izz" value="0.0314"/>
-  <xacro:property name="waist_link_02_ixx" value="0.1164"/>
-  <xacro:property name="waist_link_02_ixy" value="-0.0003"/>
-  <xacro:property name="waist_link_02_ixz" value="0.0021"/>
-  <xacro:property name="waist_link_02_iyy" value="0.0422"/>
-  <xacro:property name="waist_link_02_iyz" value="-0.0034"/>
-  <xacro:property name="waist_link_02_izz" value="0.0948"/>
-  <xacro:property name="r_arm_link_01_ixx" value="0.0077"/>
-  <xacro:property name="r_arm_link_01_ixy" value="0.0001"/>
-  <xacro:property name="r_arm_link_01_ixz" value="0.0"/>
-  <xacro:property name="r_arm_link_01_iyy" value="0.0065"/>
-  <xacro:property name="r_arm_link_01_iyz" value="-0.0008"/>
-  <xacro:property name="r_arm_link_01_izz" value="0.005"/>
-  <xacro:property name="r_arm_link_02_ixx" value="0.0108"/>
+  <xacro:property name="waist_link_01_ixx" value="0.094"/>
+  <xacro:property name="waist_link_01_ixy" value="-0.0002"/>
+  <xacro:property name="waist_link_01_ixz" value="-0.0001"/>
+  <xacro:property name="waist_link_01_iyy" value="0.0712"/>
+  <xacro:property name="waist_link_01_iyz" value="0.0005"/>
+  <xacro:property name="waist_link_01_izz" value="0.0565"/>
+  <xacro:property name="waist_link_02_ixx" value="0.1614"/>
+  <xacro:property name="waist_link_02_ixy" value="-0.0006"/>
+  <xacro:property name="waist_link_02_ixz" value="0.0026"/>
+  <xacro:property name="waist_link_02_iyy" value="0.0558"/>
+  <xacro:property name="waist_link_02_iyz" value="-0.0059"/>
+  <xacro:property name="waist_link_02_izz" value="0.1339"/>
+  <xacro:property name="r_arm_link_01_ixx" value="0.0092"/>
+  <xacro:property name="r_arm_link_01_ixy" value="0.0002"/>
+  <xacro:property name="r_arm_link_01_ixz" value="-0.0001"/>
+  <xacro:property name="r_arm_link_01_iyy" value="0.0077"/>
+  <xacro:property name="r_arm_link_01_iyz" value="-0.001"/>
+  <xacro:property name="r_arm_link_01_izz" value="0.006"/>
+  <xacro:property name="r_arm_link_02_ixx" value="0.0118"/>
   <xacro:property name="r_arm_link_02_ixy" value="0.0002"/>
   <xacro:property name="r_arm_link_02_ixz" value="-0.0001"/>
-  <xacro:property name="r_arm_link_02_iyy" value="0.0055"/>
+  <xacro:property name="r_arm_link_02_iyy" value="0.006"/>
   <xacro:property name="r_arm_link_02_iyz" value="-0.0001"/>
-  <xacro:property name="r_arm_link_02_izz" value="0.0116"/>
-  <xacro:property name="r_arm_link_03_ixx" value="0.0138"/>
+  <xacro:property name="r_arm_link_02_izz" value="0.0127"/>
+  <xacro:property name="r_arm_link_03_ixx" value="0.0143"/>
   <xacro:property name="r_arm_link_03_ixy" value="0.0"/>
-  <xacro:property name="r_arm_link_03_ixz" value="-0.0011"/>
-  <xacro:property name="r_arm_link_03_iyy" value="0.0153"/>
+  <xacro:property name="r_arm_link_03_ixz" value="-0.0001"/>
+  <xacro:property name="r_arm_link_03_iyy" value="0.016"/>
   <xacro:property name="r_arm_link_03_iyz" value="0.0"/>
-  <xacro:property name="r_arm_link_03_izz" value="0.0037"/>
-  <xacro:property name="r_arm_link_04_ixx" value="0.0105"/>
-  <xacro:property name="r_arm_link_04_ixy" value="0.0"/>
-  <xacro:property name="r_arm_link_04_ixz" value="0.0011"/>
-  <xacro:property name="r_arm_link_04_iyy" value="0.0093"/>
+  <xacro:property name="r_arm_link_03_izz" value="0.0038"/>
+  <xacro:property name="r_arm_link_04_ixx" value="0.0123"/>
+  <xacro:property name="r_arm_link_04_ixy" value="-0.0001"/>
+  <xacro:property name="r_arm_link_04_ixz" value="0.0013"/>
+  <xacro:property name="r_arm_link_04_iyy" value="0.0109"/>
   <xacro:property name="r_arm_link_04_iyz" value="-0.0003"/>
-  <xacro:property name="r_arm_link_04_izz" value="0.0031"/>
-  <xacro:property name="r_arm_link_05_ixx" value="0.0051"/>
+  <xacro:property name="r_arm_link_04_izz" value="0.0037"/>
+  <xacro:property name="r_arm_link_05_ixx" value="0.0049"/>
   <xacro:property name="r_arm_link_05_ixy" value="-0.0001"/>
-  <xacro:property name="r_arm_link_05_ixz" value="0.0001"/>
-  <xacro:property name="r_arm_link_05_iyy" value="0.0043"/>
+  <xacro:property name="r_arm_link_05_ixz" value="-0.0004"/>
+  <xacro:property name="r_arm_link_05_iyy" value="0.0041"/>
   <xacro:property name="r_arm_link_05_iyz" value="0.0003"/>
   <xacro:property name="r_arm_link_05_izz" value="0.0023"/>
-  <xacro:property name="r_arm_link_06_ixx" value="0.0037"/>
+  <xacro:property name="r_arm_link_06_ixx" value="0.002"/>
   <xacro:property name="r_arm_link_06_ixy" value="0.0"/>
-  <xacro:property name="r_arm_link_06_ixz" value="-0.0002"/>
-  <xacro:property name="r_arm_link_06_iyy" value="0.0049"/>
+  <xacro:property name="r_arm_link_06_ixz" value="-0.0001"/>
+  <xacro:property name="r_arm_link_06_iyy" value="0.0029"/>
   <xacro:property name="r_arm_link_06_iyz" value="0.0"/>
-  <xacro:property name="r_arm_link_06_izz" value="0.0031"/>
-  <xacro:property name="r_arm_link_07_ixx" value="0.0108"/>
-  <xacro:property name="r_arm_link_07_ixy" value="0.0005"/>
-  <xacro:property name="r_arm_link_07_ixz" value="0.0003"/>
-  <xacro:property name="r_arm_link_07_iyy" value="0.0125"/>
-  <xacro:property name="r_arm_link_07_iyz" value="-0.0004"/>
-  <xacro:property name="r_arm_link_07_izz" value="0.0033"/>
-  <xacro:property name="l_arm_link_01_ixx" value="0.0077"/>
+  <xacro:property name="r_arm_link_06_izz" value="0.0021"/>
+  <xacro:property name="r_arm_link_07_ixx" value="0.0071"/>
+  <xacro:property name="r_arm_link_07_ixy" value="0.0003"/>
+  <xacro:property name="r_arm_link_07_ixz" value="0.0002"/>
+  <xacro:property name="r_arm_link_07_iyy" value="0.0082"/>
+  <xacro:property name="r_arm_link_07_iyz" value="-0.0003"/>
+  <xacro:property name="r_arm_link_07_izz" value="0.0022"/>
+  <xacro:property name="l_arm_link_01_ixx" value="0.0092"/>
   <xacro:property name="l_arm_link_01_ixy" value="-0.0001"/>
   <xacro:property name="l_arm_link_01_ixz" value="0.0"/>
-  <xacro:property name="l_arm_link_01_iyy" value="0.0064"/>
-  <xacro:property name="l_arm_link_01_iyz" value="0.0008"/>
-  <xacro:property name="l_arm_link_01_izz" value="0.0051"/>
-  <xacro:property name="l_arm_link_02_ixx" value="0.0106"/>
+  <xacro:property name="l_arm_link_01_iyy" value="0.0077"/>
+  <xacro:property name="l_arm_link_01_iyz" value="0.001"/>
+  <xacro:property name="l_arm_link_01_izz" value="0.006"/>
+  <xacro:property name="l_arm_link_02_ixx" value="0.0116"/>
   <xacro:property name="l_arm_link_02_ixy" value="-0.0001"/>
   <xacro:property name="l_arm_link_02_ixz" value="-0.0001"/>
-  <xacro:property name="l_arm_link_02_iyy" value="0.0058"/>
+  <xacro:property name="l_arm_link_02_iyy" value="0.0063"/>
   <xacro:property name="l_arm_link_02_iyz" value="0.0001"/>
-  <xacro:property name="l_arm_link_02_izz" value="0.012"/>
-  <xacro:property name="l_arm_link_03_ixx" value="0.0138"/>
+  <xacro:property name="l_arm_link_02_izz" value="0.0131"/>
+  <xacro:property name="l_arm_link_03_ixx" value="0.0143"/>
   <xacro:property name="l_arm_link_03_ixy" value="0.0"/>
   <xacro:property name="l_arm_link_03_ixz" value="-0.0011"/>
-  <xacro:property name="l_arm_link_03_iyy" value="0.0153"/>
-  <xacro:property name="l_arm_link_03_iyz" value="0.0"/>
-  <xacro:property name="l_arm_link_03_izz" value="0.0037"/>
-  <xacro:property name="l_arm_link_04_ixx" value="0.0105"/>
+  <xacro:property name="l_arm_link_03_iyy" value="0.016"/>
+  <xacro:property name="l_arm_link_03_iyz" value="0.0001"/>
+  <xacro:property name="l_arm_link_03_izz" value="0.0038"/>
+  <xacro:property name="l_arm_link_04_ixx" value="0.0124"/>
   <xacro:property name="l_arm_link_04_ixy" value="0.0001"/>
-  <xacro:property name="l_arm_link_04_ixz" value="0.0011"/>
-  <xacro:property name="l_arm_link_04_iyy" value="0.0094"/>
-  <xacro:property name="l_arm_link_04_iyz" value="0.0002"/>
-  <xacro:property name="l_arm_link_04_izz" value="0.0031"/>
-  <xacro:property name="l_arm_link_05_ixx" value="0.0051"/>
+  <xacro:property name="l_arm_link_04_ixz" value="0.0013"/>
+  <xacro:property name="l_arm_link_04_iyy" value="0.011"/>
+  <xacro:property name="l_arm_link_04_iyz" value="0.0003"/>
+  <xacro:property name="l_arm_link_04_izz" value="0.0037"/>
+  <xacro:property name="l_arm_link_05_ixx" value="0.0049"/>
   <xacro:property name="l_arm_link_05_ixy" value="0.0001"/>
   <xacro:property name="l_arm_link_05_ixz" value="-0.0004"/>
-  <xacro:property name="l_arm_link_05_iyy" value="0.0043"/>
+  <xacro:property name="l_arm_link_05_iyy" value="0.0041"/>
   <xacro:property name="l_arm_link_05_iyz" value="-0.0004"/>
-  <xacro:property name="l_arm_link_05_izz" value="0.0024"/>
-  <xacro:property name="l_arm_link_06_ixx" value="0.0031"/>
+  <xacro:property name="l_arm_link_05_izz" value="0.0023"/>
+  <xacro:property name="l_arm_link_06_ixx" value="0.0002"/>
   <xacro:property name="l_arm_link_06_ixy" value="0.0"/>
   <xacro:property name="l_arm_link_06_ixz" value="-0.0001"/>
-  <xacro:property name="l_arm_link_06_iyy" value="0.0044"/>
+  <xacro:property name="l_arm_link_06_iyy" value="0.0028"/>
   <xacro:property name="l_arm_link_06_iyz" value="0.0"/>
-  <xacro:property name="l_arm_link_06_izz" value="0.0032"/>
-  <xacro:property name="l_arm_link_07_ixx" value="0.0017"/>
-  <xacro:property name="l_arm_link_07_ixy" value="0.0"/>
-  <xacro:property name="l_arm_link_07_ixz" value="0.0004"/>
-  <xacro:property name="l_arm_link_07_iyy" value="0.0031"/>
-  <xacro:property name="l_arm_link_07_iyz" value="0.0"/>
-  <xacro:property name="l_arm_link_07_izz" value="0.0029"/>
+  <xacro:property name="l_arm_link_06_izz" value="0.0021"/>
+  <xacro:property name="l_arm_link_07_ixx" value="0.0057"/>
+  <xacro:property name="l_arm_link_07_ixy" value="-0.0002"/>
+  <xacro:property name="l_arm_link_07_ixz" value="-0.0007"/>
+  <xacro:property name="l_arm_link_07_iyy" value="0.0072"/>
+  <xacro:property name="l_arm_link_07_iyz" value="0.0006"/>
+  <xacro:property name="l_arm_link_07_izz" value="0.0027"/>
 </robot>
