Commit message: Add Hand
Hand xacro added

File: DualArm/dualarm_description/urdf/dual_arm.xacro (robot description, xacro)
@@ -37,5 +37,5 @@
 			izz="${base_link_izz}"
 			vis_rpy="0 0 ${M_PI}"
-			vis_xyz="0 0 0"
+			vis_xyz="0 0 0.3"
 			mesh_file="package://dualarm_description/meshes/dualarm/base.STL"
 			mesh_scale="0.001 0.001 0.001"
@@ -47,5 +47,5 @@
 			axis_xyz="0 0 1"
 			origin_rpy="0 0 0"
-			origin_xyz="0 0 0.352"
+			origin_xyz="0 0 0.652"
 			parent="${base_link_name}"
 			child="${waist_link_01_name}"
@@ -59,5 +59,5 @@
 			mass="${waist_link_01_mass}"
 			origin_rpy="0 0 0"
-			origin_xyz="0 0 0.352"
+			origin_xyz="0 0 0.652"
 			ixx="${waist_link_01_ixx}"
 			ixy="${waist_link_01_ixy}"
@@ -74,5 +74,5 @@
 			name="dualarm_joint2"
 			type="revolute"
-			axis_xyz="0 1 0"
+			axis_xyz="0 -1 0"
 			origin_rpy="0 0 0"
 			origin_xyz="0 0 0.148"
@@ -80,6 +80,6 @@
 			child="${waist_link_02_name}"
 			limit_effort="800"
-			limit_lower="-${M_PI/8}"
-			limit_upper="${M_PI/2}"
+			limit_lower="-${M_PI/2}"
+			limit_upper="${M_PI/8}"
 			limit_v="1"
 	/>
@@ -104,5 +104,5 @@
 			name="dualarm_joint3"
 			type="revolute"
-			axis_xyz="0 0 1"
+			axis_xyz="0 0 -1"
 			origin_rpy="0 0 0"
 			origin_xyz="0 -0.125 0.217"
@@ -110,6 +110,6 @@
 			child="${r_arm_link_01_name}"
 			limit_effort="300"
-			limit_lower="-${M_PI/4}"
-			limit_upper="${M_PI/2}"
+			limit_lower="-${M_PI/2}"
+			limit_upper="${M_PI/4}"
 			limit_v="1"
 	/>
@@ -255,6 +255,6 @@
 			child="${r_arm_link_06_name}"
 			limit_effort="100"
-			limit_lower="-${M_PI/4}"
-			limit_upper="${M_PI/4}"
+			limit_lower="-${M_PI/2}"
+			limit_upper="${M_PI/2}"
 			limit_v="1"
 	/>
@@ -272,5 +272,34 @@
 			vis_rpy="0 0 0"
 			vis_xyz="0 0 0"
-			mesh_file="package://dualarm_description/meshes/dualarm1/link8.STL"
+			mesh_file="package://dualarm_description/meshes/dualarm1/Wrist.STL"
+			mesh_scale="0.001 0.001 0.001"
+	/>
+	<m_joint_100
+		name="dualarm_joint15"
+		type="revolute"
+		axis_xyz="1 0 0"
+		origin_rpy="0 0 0"
+		origin_xyz="0 0 -0.216"
+		parent="${r_arm_link_06_name}"
+		child="${r_arm_link_hand}"
+		limit_effort="100"
+		limit_lower="-${3*M_PI/2}"
+		limit_upper="${3*M_PI/2}"
+		limit_v="1"
+	/>
+	<m_link_cylinder
+			name="${r_arm_link_hand}"
+			mass="${r_arm_link_07_mass}"
+			origin_rpy="0 0 0"
+			origin_xyz="0 0 -0.216"
+			ixx="${r_arm_link_07_ixx}"
+			ixy="${r_arm_link_07_ixy}"
+			ixz="${r_arm_link_07_ixz}"
+			iyy="${r_arm_link_07_iyy}"
+			iyz="${r_arm_link_07_iyz}"
+			izz="${r_arm_link_07_izz}"
+			vis_rpy="0 0 0"
+			vis_xyz="0 0 0"
+			mesh_file="package://dualarm_description/meshes/dualarm1/Hand.STL"
 			mesh_scale="0.001 0.001 0.001"
 	/>
@@ -279,5 +308,5 @@
 			name="dualarm_joint9"
 			type="revolute"
-			axis_xyz="0 0 1"
+			axis_xyz="0 0 -1"
 			origin_rpy="0 0 0"
 			origin_xyz="0 0.125 0.217"
@@ -285,6 +314,6 @@
 			child="${l_arm_link_01_name}"
 			limit_effort="300"
-			limit_lower="-${M_PI/2}"
-			limit_upper="${M_PI/4}"
+			limit_lower="-${M_PI/4}"
+			limit_upper="${M_PI/2}"
 			limit_v="1"
 	/>
@@ -308,5 +337,5 @@
 			name="dualarm_joint10"
 			type="revolute"
-			axis_xyz="0 1 0"
+			axis_xyz="0 -1 0"
 			origin_rpy="0 0 0"
 			origin_xyz="0 0.09 0.083"
@@ -395,5 +424,5 @@
 			name="dualarm_joint13"
 			type="revolute"
-			axis_xyz="0 1 0"
+			axis_xyz="0 -1 0"
 			origin_rpy="0 0 0"
 			origin_xyz="-0.0245 0 -0.158"
@@ -401,6 +430,6 @@
 			child="${l_arm_link_05_name}"
 			limit_effort="100"
-			limit_lower="-${M_PI/2}"
-			limit_upper="${M_PI/4}"
+			limit_lower="-${M_PI/4}"
+			limit_upper="${M_PI/2}"
 			limit_v="1"
 	/>
@@ -428,12 +457,12 @@
 			origin_xyz="0.0245 0 -0.155"
 			parent="${l_arm_link_05_name}"
-			child="${l_arm_link_06_name}"
+			child="${l_arm_link_hand}"
 			limit_effort="100"
-			limit_lower="-${M_PI/4}"
-			limit_upper="${M_PI/4}"
-			limit_v="1"
-	/>
-	<m_link_cylinder
-			name="${l_arm_link_06_name}"
+			limit_lower="-${3*M_PI/2}"
+			limit_upper="${3*M_PI/2}"
+			limit_v="1"
+	/>
+	<m_link_cylinder
+			name="${l_arm_link_hand}"
 			mass="${l_arm_link_06_mass}"
 			origin_rpy="0 0 0"
@@ -447,5 +476,5 @@
 			vis_rpy="0 0 0"
 			vis_xyz="0 0 0"
-			mesh_file="package://dualarm_description/meshes/dualarm1/link8.STL"
+			mesh_file="package://dualarm_description/meshes/dualarm1/HandwithWrist.STL"
 			mesh_scale="0.001 0.001 0.001"
 	/>

File: DualArm/dualarm_description/urdf/robot_parameter.xacro (robot description, xacro)
@@ -14,4 +14,5 @@
   <xacro:property name="r_arm_link_05_name" value="link_07" />
   <xacro:property name="r_arm_link_06_name" value="link_08" />
+  <xacro:property name="r_arm_link_hand" value="link_R_hand" />
 <!--left_arm-->
   <xacro:property name="l_arm_link_01_name" value="link_09" />
@@ -20,5 +21,5 @@
   <xacro:property name="l_arm_link_04_name" value="link_12" />
   <xacro:property name="l_arm_link_05_name" value="link_13" />
-  <xacro:property name="l_arm_link_06_name" value="link_14" />
+  <xacro:property name="l_arm_link_hand" value="link_L_hand" />
 <!-- link_mass -->
   <xacro:property name="base_link_mass" value="10.0"/>
@@ -30,5 +31,6 @@
   <xacro:property name="r_arm_link_04_mass" value="2.49"/>
   <xacro:property name="r_arm_link_05_mass" value="1.86"/>
-  <xacro:property name="r_arm_link_06_mass" value="0.0646"/>
+  <xacro:property name="r_arm_link_06_mass" value="2.676"/>
+  <xacro:property name="r_arm_link_07_mass" value="1.29"/>
   <xacro:property name="l_arm_link_01_mass" value="3.35"/>
   <xacro:property name="l_arm_link_02_mass" value="3.51"/>
@@ -36,5 +38,5 @@
   <xacro:property name="l_arm_link_04_mass" value="2.49"/>
   <xacro:property name="l_arm_link_05_mass" value="1.86"/>
-  <xacro:property name="l_arm_link_06_mass" value="0.0646"/>
+  <xacro:property name="l_arm_link_06_mass" value="2.1946"/>
 <!-- link_inertia -->
   <xacro:property name="base_link_ixx" value="0.0"/>
@@ -86,10 +88,16 @@
   <xacro:property name="r_arm_link_05_iyz" value="298769.64E-9"/>
   <xacro:property name="r_arm_link_05_izz" value="2250292.68E-9"/>
-  <xacro:property name="r_arm_link_06_ixx" value="0.00005"/>
+  <xacro:property name="r_arm_link_06_ixx" value="15715348.78E-9"/>
   <xacro:property name="r_arm_link_06_ixy" value="0.0"/>
-  <xacro:property name="r_arm_link_06_ixz" value="0.0"/>
-  <xacro:property name="r_arm_link_06_iyy" value="0.00005"/>
+  <xacro:property name="r_arm_link_06_ixz" value="-347842.21E-9"/>
+  <xacro:property name="r_arm_link_06_iyy" value="16761167.93E-9"/>
   <xacro:property name="r_arm_link_06_iyz" value="0.0"/>
-  <xacro:property name="r_arm_link_06_izz" value="0.00005"/>
+  <xacro:property name="r_arm_link_06_izz" value="3543832.43E-9"/>
+  <xacro:property name="r_arm_link_07_ixx" value="7534883.39E-9"/>
+  <xacro:property name="r_arm_link_07_ixy" value="0.0"/>
+  <xacro:property name="r_arm_link_07_ixz" value="0.0"/>
+  <xacro:property name="r_arm_link_07_iyy" value="9485578.12E-9"/>
+  <xacro:property name="r_arm_link_07_iyz" value="-659219.99E-9"/>
+  <xacro:property name="r_arm_link_07_izz" value="25880996.64E-9"/>
   <xacro:property name="l_arm_link_01_ixx" value="0.0057"/>
   <xacro:property name="l_arm_link_01_ixy" value="0.0"/>
@@ -122,9 +130,9 @@
   <xacro:property name="l_arm_link_05_iyz" value="-355897.62E-9"/>
   <xacro:property name="l_arm_link_05_izz" value="2255248.43E-9"/>
-  <xacro:property name="l_arm_link_06_ixx" value="0.00005"/>
-  <xacro:property name="l_arm_link_06_ixy" value="0.0"/>
-  <xacro:property name="l_arm_link_06_ixz" value="0.0"/>
-  <xacro:property name="l_arm_link_06_iyy" value="0.00005"/>
-  <xacro:property name="l_arm_link_06_iyz" value="0.0"/>
-  <xacro:property name="l_arm_link_06_izz" value="0.00005"/>
+  <xacro:property name="l_arm_link_06_ixx" value="64638829.47E-9"/>
+  <xacro:property name="l_arm_link_06_ixy" value="-182585.55E-9"/>
+  <xacro:property name="l_arm_link_06_ixz" value="-1132418.18E-9"/>
+  <xacro:property name="l_arm_link_06_iyy" value="66659017.77E-9"/>
+  <xacro:property name="l_arm_link_06_iyz" value="2023270.8E-9"/>
+  <xacro:property name="l_arm_link_06_izz" value="4566899.4E-9"/>
 </robot>

Commit message: Version 20.09.16
16-dof update

File: DualArm/dualarm_description/urdf/dual_arm.xacro (robot description, xacro)
@@ -3,5 +3,5 @@
 	<xacro:include filename="$(find dualarm_description)/urdf/link_to_joint.xacro" />
 	<xacro:include filename="$(find dualarm_description)/urdf/robot_parameter.xacro" />
-	<xacro:include filename="$(find dualarm_description)/urdf/dual_arm.gazebo.xacro" />
+	<xacro:include filename="$(find dualarm_description)/urdf/dual_arm.gazebo" />
 	<!-- Base parts -->
 	<link name = "world"/>
@@ -29,5 +29,5 @@
 			mass="${base_link_mass}"
 			origin_rpy= "0 0 0"
-			origin_xyz="0 0 0"
+			origin_xyz="0 0 0.3"
 			ixx="${base_link_ixx}"
 			ixy="${base_link_ixy}"
@@ -47,5 +47,5 @@
 			axis_xyz="0 0 1"
 			origin_rpy="0 0 0"
-			origin_xyz="0 0 0.658"
+			origin_xyz="0 0 0.652"
 			parent="${base_link_name}"
 			child="${waist_link_01_name}"
@@ -67,5 +67,5 @@
 			izz="${waist_link_01_izz}"
 			vis_rpy="0 0 0"
-			vis_xyz="0 0 0.0"
+			vis_xyz="0 0 -0.011"
 			mesh_file="package://dualarm_description/meshes/dualarm1/link1.STL"
 			mesh_scale="0.001 0.001 0.001"
@@ -155,5 +155,5 @@
 			izz="${r_arm_link_02_izz}"
 			vis_rpy="0 0 0"
-			vis_xyz="0 0 0"
+			vis_xyz="0 0.011 0"
 			mesh_file="package://dualarm_description/meshes/dualarm1/link4.STL"
 			mesh_scale="0.001 0.001 0.001"
@@ -193,5 +193,5 @@
 			axis_xyz="0 0 1"
 			origin_rpy="0 0 0"
-			origin_xyz="0 0 -0.158"
+			origin_xyz="0 0 -0.242"
 			parent="${r_arm_link_03_name}"
 			child="${r_arm_link_04_name}"
@@ -280,5 +280,5 @@
 		axis_xyz="1 0 0"
 		origin_rpy="0 0 0"
-		origin_xyz="0 0 -0.216"
+		origin_xyz="0 0 -0.066"
 		parent="${r_arm_link_06_name}"
 		child="${r_arm_link_hand}"
@@ -292,5 +292,5 @@
 			mass="${r_arm_link_07_mass}"
 			origin_rpy="0 0 0"
-			origin_xyz="0.01382 0.01787 -0.12277"
+			origin_xyz="0 0 0"
 			ixx="${r_arm_link_07_ixx}"
 			ixy="${r_arm_link_07_ixy}"
@@ -301,5 +301,5 @@
 			vis_rpy="0 0 0"
 			vis_xyz="0 0 0"
-			mesh_file="package://dualarm_description/meshes/dualarm1/Hand.STL"
+			mesh_file="package://dualarm_description/meshes/dualarm1/Allegro_wrist.STL"
 			mesh_scale="0.001 0.001 0.001"
 	/>
@@ -359,5 +359,5 @@
 			izz="${l_arm_link_02_izz}"
 			vis_rpy="${M_PI} 0 0"
-			vis_xyz="0 0 0"
+			vis_xyz="0 -0.011 0"
 			mesh_file="package://dualarm_description/meshes/dualarm1/link4.STL"
 			mesh_scale="0.001 0.001 0.001"
@@ -397,5 +397,5 @@
 			axis_xyz="0 0 1"
 			origin_rpy="0 0 0"
-			origin_xyz="0 0 -0.158"
+			origin_xyz="0 0 -0.242"
 			parent="${l_arm_link_03_name}"
 			child="${l_arm_link_04_name}"
@@ -457,5 +457,5 @@
 			origin_xyz="0.0245 0 -0.155"
 			parent="${l_arm_link_05_name}"
-			child="${l_arm_link_hand}"
+			child="${l_arm_link_06_name}"
 			limit_effort="100"
 			limit_lower="-${3*M_PI/2}"
@@ -464,8 +464,8 @@
 	/>
 	<m_link_cylinder
-			name="${l_arm_link_hand}"
+			name="${l_arm_link_06_name}"
 			mass="${l_arm_link_06_mass}"
 			origin_rpy="0 0 0"
-			origin_xyz="0.00824 -0.01572 -0.19016"
+			origin_xyz="0 0 0"
 			ixx="${l_arm_link_06_ixx}"
 			ixy="${l_arm_link_06_ixy}"
@@ -476,5 +476,34 @@
 			vis_rpy="0 0 0"
 			vis_xyz="0 0 0"
-			mesh_file="package://dualarm_description/meshes/dualarm1/HandwithWrist.STL"
+			mesh_file="package://dualarm_description/meshes/dualarm1/Wrist_controller.STL"
+			mesh_scale="0.001 0.001 0.001"
+	/>
+	<m_joint_100
+			name="dualarm_joint16"
+			type="revolute"
+			axis_xyz="0 0 1"
+			origin_rpy="0 0 0"
+			origin_xyz="0 0 -0.205"
+			parent="${l_arm_link_06_name}"
+			child="${l_arm_link_hand}"
+			limit_effort="100"
+			limit_lower="-${3*M_PI/2}"
+			limit_upper="${3*M_PI/2}"
+			limit_v="1"
+	/>
+	<m_link_cylinder
+			name="${l_arm_link_hand}"
+			mass="${l_arm_link_07_mass}"
+			origin_rpy="0 0 0"
+			origin_xyz="0 0 0"
+			ixx="${l_arm_link_07_ixx}"
+			ixy="${l_arm_link_07_ixy}"
+			ixz="${l_arm_link_07_ixz}"
+			iyy="${l_arm_link_07_iyy}"
+			iyz="${l_arm_link_07_iyz}"
+			izz="${l_arm_link_07_izz}"
+			vis_rpy="0 0 0"
+			vis_xyz="0 0 0"
+			mesh_file="package://dualarm_description/meshes/dualarm1/hand_adapter_L.STL"
 			mesh_scale="0.001 0.001 0.001"
 	/>

File: DualArm/dualarm_description/urdf/robot_parameter.xacro (robot description, xacro)
@@ -21,4 +21,5 @@
   <xacro:property name="l_arm_link_04_name" value="link_12" />
   <xacro:property name="l_arm_link_05_name" value="link_13" />
+  <xacro:property name="l_arm_link_06_name" value="link_14" />
   <xacro:property name="l_arm_link_hand" value="link_L_hand" />
 <!-- link_mass -->
@@ -39,4 +40,5 @@
   <xacro:property name="l_arm_link_05_mass" value="1.86"/>
   <xacro:property name="l_arm_link_06_mass" value="2.1946"/>
+  <xacro:property name="l_arm_link_07_mass" value="1.29"/>
 <!-- link_inertia -->
   <xacro:property name="base_link_ixx" value="0.0"/>
@@ -46,10 +48,10 @@
   <xacro:property name="base_link_izz" value="0.0"/>
   <xacro:property name="base_link_iyz" value="0.0"/>
-  <xacro:property name="waist_link_01_ixx" value="83854563.43E-9"/>
-  <xacro:property name="waist_link_01_ixy" value="-135841.54E-9"/>
-  <xacro:property name="waist_link_01_ixz" value="-625787.35E-9"/>
-  <xacro:property name="waist_link_01_iyy" value="70969371.34E-9"/>
-  <xacro:property name="waist_link_01_iyz" value="-15432807.98E-9"/>
-  <xacro:property name="waist_link_01_izz" value="53062013.96E-9"/>
+  <xacro:property name="waist_link_01_ixx" value="0.0463"/>
+  <xacro:property name="waist_link_01_ixy" value="0.0"/>
+  <xacro:property name="waist_link_01_ixz" value="0.0"/>
+  <xacro:property name="waist_link_01_iyy" value="-0.0637"/>
+  <xacro:property name="waist_link_01_iyz" value="0.0027"/>
+  <xacro:property name="waist_link_01_izz" value="0.0271"/>
   <xacro:property name="waist_link_02_ixx" value="0.1408"/>
   <xacro:property name="waist_link_02_ixy" value="0.0"/>
@@ -88,10 +90,10 @@
   <xacro:property name="r_arm_link_05_iyz" value="298769.64E-9"/>
   <xacro:property name="r_arm_link_05_izz" value="2250292.68E-9"/>
-  <xacro:property name="r_arm_link_06_ixx" value="15715348.78E-9"/>
-  <xacro:property name="r_arm_link_06_ixy" value="0.0"/>
-  <xacro:property name="r_arm_link_06_ixz" value="-347842.21E-9"/>
-  <xacro:property name="r_arm_link_06_iyy" value="16761167.93E-9"/>
-  <xacro:property name="r_arm_link_06_iyz" value="0.0"/>
-  <xacro:property name="r_arm_link_06_izz" value="3543832.43E-9"/>
+  <xacro:property name="r_arm_link_06_ixx" value="372762541.12E-9"/>
+  <xacro:property name="r_arm_link_06_ixy" value="-3411073.92E-9"/>
+  <xacro:property name="r_arm_link_06_ixz" value="1777052.78E-9"/>
+  <xacro:property name="r_arm_link_06_iyy" value="91135956.07E-9"/>
+  <xacro:property name="r_arm_link_06_iyz" value="-156654091.62E-9"/>
+  <xacro:property name="r_arm_link_06_izz" value="3212626.70E-9"/>
   <xacro:property name="r_arm_link_07_ixx" value="7534883.39E-9"/>
   <xacro:property name="r_arm_link_07_ixy" value="0.0"/>
@@ -136,3 +138,9 @@
   <xacro:property name="l_arm_link_06_iyz" value="2023270.8E-9"/>
   <xacro:property name="l_arm_link_06_izz" value="4566899.4E-9"/>
+  <xacro:property name="l_arm_link_07_ixx" value="7534883.39E-9"/>
+  <xacro:property name="l_arm_link_07_ixy" value="0.0"/>
+  <xacro:property name="l_arm_link_07_ixz" value="0.0"/>
+  <xacro:property name="l_arm_link_07_iyy" value="9485578.12E-9"/>
+  <xacro:property name="l_arm_link_07_iyz" value="-659219.99E-9"/>
+  <xacro:property name="l_arm_link_07_izz" value="25880996.64E-9"/>
 </robot>

Commit message: Version 20.10.25
Task controller

File: DualArm/dualarm_description/urdf/dual_arm.xacro (robot description, xacro)
@@ -29,5 +29,5 @@
 			mass="${base_link_mass}"
 			origin_rpy= "0 0 0"
-			origin_xyz="0 0 0.3"
+			origin_xyz="0 0 0"
 			ixx="${base_link_ixx}"
 			ixy="${base_link_ixy}"
@@ -45,5 +45,5 @@
 			name="dualarm_joint1"
 			type="revolute"
-			axis_xyz="0 0 1"
+			axis_xyz="0 0 -1"
 			origin_rpy="0 0 0"
 			origin_xyz="0 0 0.652"
@@ -225,5 +225,5 @@
 			parent="${r_arm_link_04_name}"
 			child="${r_arm_link_05_name}"
-			limit_effort="100"
+			limit_effort="300"
 			limit_lower="-${M_PI/2}"
 			limit_upper="${M_PI/8}"
@@ -254,5 +254,5 @@
 			parent="${r_arm_link_05_name}"
 			child="${r_arm_link_06_name}"
-			limit_effort="100"
+			limit_effort="300"
 			limit_lower="-${M_PI}"
 			limit_upper="${M_PI}"
@@ -276,15 +276,15 @@
 	/>
 	<m_joint_100
-		name="dualarm_joint15"
-		type="revolute"
-		axis_xyz="1 0 0"
-		origin_rpy="0 0 0"
-		origin_xyz="0 0 -0.066"
-		parent="${r_arm_link_06_name}"
-		child="${r_arm_link_hand}"
-		limit_effort="100"
-		limit_lower="-${3*M_PI/2}"
-		limit_upper="${3*M_PI/2}"
-		limit_v="1"
+			name="dualarm_joint9"
+			type="revolute"
+			axis_xyz="1 0 0"
+			origin_rpy="0 0 0"
+			origin_xyz="0 0 -0.0755"
+			parent="${r_arm_link_06_name}"
+			child="${r_arm_link_hand}"
+			limit_effort="300"
+			limit_lower="-${M_PI}"
+			limit_upper="${M_PI}"
+			limit_v="1"
 	/>
 	<m_link_cylinder
@@ -304,7 +304,14 @@
 			mesh_scale="0.001 0.001 0.001"
 	/>
+	<joint name="dualarm_R_end" type="fixed">
+		<origin xyz="0 0 -0.122"
+				rpy="0 0 0"/>
+		<parent link="${r_arm_link_hand}"/>
+		<child link="dualarm_R_end_frame" />
+	</joint>
+	<link name="dualarm_R_end_frame"/>
 	<!-- left_arm part-->
 	<m_joint_100
-			name="dualarm_joint9"
+			name="dualarm_joint10"
 			type="revolute"
 			axis_xyz="0 0 -1"
@@ -335,5 +342,5 @@
 	/>
 	<m_joint_100
-			name="dualarm_joint10"
+			name="dualarm_joint11"
 			type="revolute"
 			axis_xyz="0 -1 0"
@@ -364,5 +371,5 @@
 	/>
 	<m_joint_100
-			name="dualarm_joint11"
+			name="dualarm_joint12"
 			type="revolute"
 			axis_xyz="1 0 0"
@@ -393,5 +400,5 @@
 	/>
 	<m_joint_100
-			name="dualarm_joint12"
+			name="dualarm_joint13"
 			type="revolute"
 			axis_xyz="0 0 1"
@@ -422,5 +429,5 @@
 	/>
 	<m_joint_100
-			name="dualarm_joint13"
+			name="dualarm_joint14"
 			type="revolute"
 			axis_xyz="0 -1 0"
@@ -429,5 +436,5 @@
 			parent="${l_arm_link_04_name}"
 			child="${l_arm_link_05_name}"
-			limit_effort="100"
+			limit_effort="300"
 			limit_lower="-${M_PI/4}"
 			limit_upper="${M_PI/2}"
@@ -451,5 +458,5 @@
 	/>
 	<m_joint_100
-			name="dualarm_joint14"
+			name="dualarm_joint15"
 			type="revolute"
 			axis_xyz="0 0 1"
@@ -458,7 +465,7 @@
 			parent="${l_arm_link_05_name}"
 			child="${l_arm_link_06_name}"
-			limit_effort="100"
-			limit_lower="-${3*M_PI/2}"
-			limit_upper="${3*M_PI/2}"
+			limit_effort="300"
+			limit_lower="-${M_PI}"
+			limit_upper="${M_PI}"
 			limit_v="1"
 	/>
@@ -467,5 +474,5 @@
 			mass="${l_arm_link_06_mass}"
 			origin_rpy="0 0 0"
-			origin_xyz="0 0 0"
+			origin_xyz="0.00173 0.00014 -0.13722"
 			ixx="${l_arm_link_06_ixx}"
 			ixy="${l_arm_link_06_ixy}"
@@ -476,5 +483,5 @@
 			vis_rpy="0 0 0"
 			vis_xyz="0 0 0"
-			mesh_file="package://dualarm_description/meshes/dualarm1/Wrist_controller.STL"
+			mesh_file="package://dualarm_description/meshes/dualarm1/Wrist.STL"
 			mesh_scale="0.001 0.001 0.001"
 	/>
@@ -482,12 +489,12 @@
 			name="dualarm_joint16"
 			type="revolute"
-			axis_xyz="0 0 1"
-			origin_rpy="0 0 0"
-			origin_xyz="0 0 -0.205"
+			axis_xyz="1 0 0"
+			origin_rpy="0 0 0"
+			origin_xyz="0 0 -0.0755"
 			parent="${l_arm_link_06_name}"
 			child="${l_arm_link_hand}"
-			limit_effort="100"
-			limit_lower="-${3*M_PI/2}"
-			limit_upper="${3*M_PI/2}"
+			limit_effort="300"
+			limit_lower="-${M_PI}"
+			limit_upper="${M_PI}"
 			limit_v="1"
 	/>
@@ -508,3 +515,10 @@
 			mesh_scale="0.001 0.001 0.001"
 	/>
+	<joint name="dualarm_L_end" type="fixed">
+		<origin xyz="0 0 -0.122"
+				rpy="0 0 0"/>
+		<parent link="${l_arm_link_hand}"/>
+		<child link="dualarm_L_end_frame" />
+	</joint>
+	<link name="dualarm_L_end_frame"/>
 </robot>

File: DualArm/dualarm_description/urdf/robot_parameter.xacro (robot description, xacro)
@@ -1,5 +1,5 @@
 <?xml version="1.0" ?>
 <robot xmlns:xacro="http://www.ros.org/wiki/xacro">
-  <xacro:property name="M_PI" value="3.14159"/>
+  <xacro:property name="M_PI" value="3.141592"/>
 <!--base-->
   <xacro:property name="base_link_name" value="base_link" />
@@ -16,10 +16,10 @@
   <xacro:property name="r_arm_link_hand" value="link_R_hand" />
 <!--left_arm-->
-  <xacro:property name="l_arm_link_01_name" value="link_09" />
-  <xacro:property name="l_arm_link_02_name" value="link_10" />
-  <xacro:property name="l_arm_link_03_name" value="link_11" />
-  <xacro:property name="l_arm_link_04_name" value="link_12" />
-  <xacro:property name="l_arm_link_05_name" value="link_13" />
-  <xacro:property name="l_arm_link_06_name" value="link_14" />
+  <xacro:property name="l_arm_link_01_name" value="link_10" />
+  <xacro:property name="l_arm_link_02_name" value="link_11" />
+  <xacro:property name="l_arm_link_03_name" value="link_12" />
+  <xacro:property name="l_arm_link_04_name" value="link_13" />
+  <xacro:property name="l_arm_link_05_name" value="link_14" />
+  <xacro:property name="l_arm_link_06_name" value="link_15" />
   <xacro:property name="l_arm_link_hand" value="link_L_hand" />
 <!-- link_mass -->
@@ -48,10 +48,10 @@
   <xacro:property name="base_link_izz" value="0.0"/>
   <xacro:property name="base_link_iyz" value="0.0"/>
-  <xacro:property name="waist_link_01_ixx" value="0.0463"/>
-  <xacro:property name="waist_link_01_ixy" value="0.0"/>
-  <xacro:property name="waist_link_01_ixz" value="0.0"/>
-  <xacro:property name="waist_link_01_iyy" value="-0.0637"/>
-  <xacro:property name="waist_link_01_iyz" value="0.0027"/>
-  <xacro:property name="waist_link_01_izz" value="0.0271"/>
+  <xacro:property name="waist_link_01_ixx" value="83854563.43e-9"/>
+  <xacro:property name="waist_link_01_ixy" value="-135841.54e-9"/>
+  <xacro:property name="waist_link_01_ixz" value="-625787.35e-9"/>
+  <xacro:property name="waist_link_01_iyy" value="70969371.34e-9"/>
+  <xacro:property name="waist_link_01_iyz" value="-15432807.98e-9"/>
+  <xacro:property name="waist_link_01_izz" value="53062013.96e-9"/>
   <xacro:property name="waist_link_02_ixx" value="0.1408"/>
   <xacro:property name="waist_link_02_ixy" value="0.0"/>
