Commit message: #8-1 model update
ft sensor update

File: DualArm/dualarm_description/urdf/dual_arm.gazebo.xacro (robot description, xacro)
@@ -9,3 +9,23 @@
     </plugin>
   </gazebo>
+  <gazebo reference="ft_sensor_joint_R">
+    <provideFeedback>true</provideFeedback>
+  </gazebo>
+  <gazebo>
+    <plugin name="ft_sensor" filename="libgazebo_ros_ft_sensor.so">
+      <updateRate>900</updateRate>
+      <topicName>ft_sensor_topic_R</topicName>
+      <jointName>ft_sensor_joint_R</jointName>
+    </plugin>
+  </gazebo>
+  <gazebo reference="ft_sensor_joint_L">
+    <provideFeedback>true</provideFeedback>
+  </gazebo>
+  <gazebo>
+    <plugin name="ft_sensor" filename="libgazebo_ros_ft_sensor.so">
+      <updateRate>900</updateRate>
+      <topicName>ft_sensor_topic_L</topicName>
+      <jointName>ft_sensor_joint_L</jointName>
+    </plugin>
+  </gazebo>
 </robot>

File: DualArm/dualarm_description/urdf/dual_arm.xacro (robot description, xacro)
@@ -495,5 +495,5 @@
 		<origin
 				rpy="0 0 0"
-				xyz="0 0 -0.091" />
+				xyz="0 0 -0.081" />
 		<parent
 				link="${r_arm_link_06_name}" />
@@ -542,5 +542,5 @@
 	<joint name="dualarm_R_end" type="fixed">
 		<origin
-				xyz="0 0 -0.04681"
+				xyz="0 0 -0.167"
 				rpy="0 0 0"/>
 		<parent link="${r_arm_link_hand}"/>
@@ -882,5 +882,5 @@
 		<origin
 				rpy="0 0 0"
-				xyz="0 0 -0.091" />
+				xyz="0 0 -0.081" />
 		<parent
 				link="${l_arm_link_06_name}" />
@@ -922,5 +922,5 @@
 			<geometry>
 				<mesh
-						filename="package://dualarm_description/meshes/stl/hand_adapter_L.STL"
+						filename="package://dualarm_description/meshes/stl/l7.STL"
 						scale="0.001 0.001 0.001"/>
 			</geometry>
@@ -929,5 +929,5 @@
 	<joint name="dualarm_L_end" type="fixed">
 		<origin
-				xyz="0 0 -0.04681"
+				xyz="0 0 -0.167"
 				rpy="0 0 0"/>
 		<parent link="${l_arm_link_hand}"/>

File: DualArm/dualarm_description/urdf/robot_parameter.xacro (robot description, xacro)
@@ -15,4 +15,6 @@
   <xacro:property name="r_arm_link_06_name" value="link_08" />
   <xacro:property name="r_arm_link_hand" value="link_R_hand" />
+  <xacro:property name="r_arm_link_hand_1" value="link_R_hand_1" />
+  <xacro:property name="r_arm_link_hand_2" value="link_R_hand_2" />
 <!--left_arm-->
   <xacro:property name="l_arm_link_01_name" value="link_10" />
@@ -23,4 +25,6 @@
   <xacro:property name="l_arm_link_06_name" value="link_15" />
   <xacro:property name="l_arm_link_hand" value="link_L_hand" />
+  <xacro:property name="l_arm_link_hand_1" value="link_L_hand_1" />
+  <xacro:property name="l_arm_link_hand_2" value="link_L_hand_2" />
 <!-- link_mass -->
   <xacro:property name="base_link_mass" value="10.0"/>
@@ -33,5 +37,7 @@
   <xacro:property name="r_arm_link_05_mass" value="1.8"/>
   <xacro:property name="r_arm_link_06_mass" value="1.73"/>
-  <xacro:property name="r_arm_link_07_mass" value="1.08"/>
+  <xacro:property name="r_arm_link_07_mass" value="1.60"/>
+  <xacro:property name="r_arm_link_07_1_mass" value="0.50"/>
+  <xacro:property name="r_arm_link_07_2_mass" value="1.10"/>
   <xacro:property name="l_arm_link_01_mass" value="3.35"/>
   <xacro:property name="l_arm_link_02_mass" value="3.51"/>
@@ -41,4 +47,6 @@
   <xacro:property name="l_arm_link_06_mass" value="1.73"/>
   <xacro:property name="l_arm_link_07_mass" value="1.147"/>
+  <xacro:property name="l_arm_link_07_1_mass" value="0.50"/>
+  <xacro:property name="l_arm_link_07_2_mass" value="0.65"/>
 <!-- link_inertia -->
   <xacro:property name="base_link_ixx" value="0.0"/>
@@ -102,4 +110,16 @@
   <xacro:property name="r_arm_link_07_iyz" value="-0.0003"/>
   <xacro:property name="r_arm_link_07_izz" value="0.0022"/>
+  <xacro:property name="r_arm_link_07_1_ixx" value="0.0006"/>
+  <xacro:property name="r_arm_link_07_1_ixy" value="0.0"/>
+  <xacro:property name="r_arm_link_07_1_ixz" value="0.0002"/>
+  <xacro:property name="r_arm_link_07_1_iyy" value="0.0009"/>
+  <xacro:property name="r_arm_link_07_1_iyz" value="0.0"/>
+  <xacro:property name="r_arm_link_07_1_izz" value="0.0009"/>
+  <xacro:property name="r_arm_link_07_2_ixx" value="0.0056"/>
+  <xacro:property name="r_arm_link_07_2_ixy" value="0.0005"/>
+  <xacro:property name="r_arm_link_07_2_ixz" value="0.0008"/>
+  <xacro:property name="r_arm_link_07_2_iyy" value="0.007"/>
+  <xacro:property name="r_arm_link_07_2_iyz" value="0.0002"/>
+  <xacro:property name="r_arm_link_07_2_izz" value="0.0023"/>
   <xacro:property name="l_arm_link_01_ixx" value="0.0092"/>
   <xacro:property name="l_arm_link_01_ixy" value="-0.0001"/>
@@ -144,3 +164,15 @@
   <xacro:property name="l_arm_link_07_iyz" value="0.0006"/>
   <xacro:property name="l_arm_link_07_izz" value="0.0027"/>
+  <xacro:property name="l_arm_link_07_1_ixx" value="0.0006"/>
+  <xacro:property name="l_arm_link_07_1_ixy" value="0.0"/>
+  <xacro:property name="l_arm_link_07_1_ixz" value="0.0001"/>
+  <xacro:property name="l_arm_link_07_1_iyy" value="0.0010"/>
+  <xacro:property name="l_arm_link_07_1_iyz" value="0.0"/>
+  <xacro:property name="l_arm_link_07_1_izz" value="0.0009"/>
+  <xacro:property name="l_arm_link_07_2_ixx" value="0.0025"/>
+  <xacro:property name="l_arm_link_07_2_ixy" value="0.0000"/>
+  <xacro:property name="l_arm_link_07_2_ixz" value="-0.0001"/>
+  <xacro:property name="l_arm_link_07_2_iyy" value="0.0037"/>
+  <xacro:property name="l_arm_link_07_2_iyz" value="0.0000"/>
+  <xacro:property name="l_arm_link_07_2_izz" value="0.0014"/>
 </robot>

Commit message: #9 model update
ft sensor test done

File: DualArm/dualarm_description/urdf/dual_arm.gazebo.xacro (robot description, xacro)
@@ -11,4 +11,6 @@
   <gazebo reference="ft_sensor_joint_R">
     <provideFeedback>true</provideFeedback>
+    <disableFixedJointLumping>true</disableFixedJointLumping>
+    <preserveFixedJoint>true</preserveFixedJoint>
   </gazebo>
   <gazebo>
@@ -21,4 +23,6 @@
   <gazebo reference="ft_sensor_joint_L">
     <provideFeedback>true</provideFeedback>
+    <disableFixedJointLumping>true</disableFixedJointLumping>
+    <preserveFixedJoint>true</preserveFixedJoint>
   </gazebo>
   <gazebo>

File: DualArm/dualarm_description/urdf/dual_arm1.xacro (robot description, xacro)
@@ -540,5 +540,5 @@
 		</visual>
 	</link>
-	<joint name="ft_sensor_joint_R" type="revolute">
+	<joint name="ft_sensor_joint_R" type="fixed">
 		<parent link="${r_arm_link_hand_1}"/>
 		<child link="${r_arm_link_hand_2}"/>
@@ -546,5 +546,5 @@
 				rpy="0 0 0"
 				xyz="0 0 -0.057"/>
-		<limit effort="100" velocity="100" lower="0" upper="0"/>
+		<limit effort="1000" velocity="100" lower="0" upper="0"/>
 	</joint>
 	<link name="${r_arm_link_hand_2}">
@@ -960,5 +960,5 @@
 		</visual>
 	</link>
-	<joint name="ft_sensor_joint_L" type="revolute">
+	<joint name="ft_sensor_joint_L" type="fixed">
 		<parent link="${l_arm_link_hand_1}"/>
 		<child link="${l_arm_link_hand_2}"/>
@@ -966,5 +966,5 @@
 				rpy="0 0 0"
 				xyz="0 0 -0.057"/>
-		<limit effort="100" velocity="100" lower="0" upper="0"/>
+		<limit effort="1000" velocity="100" lower="0" upper="0"/>
 	</joint>
 	<link name="${l_arm_link_hand_2}">
