Commit message: #20 dissertation

File: DualArm/dualarm_description/urdf/robot_parameter.xacro (robot description, xacro)
@@ -40,5 +40,5 @@
   <xacro:property name="r_arm_link_07_mass" value="1.60"/>
   <xacro:property name="r_arm_link_07_1_mass" value="0.50"/>
-  <xacro:property name="r_arm_link_07_2_mass" value="1.10"/>
+  <xacro:property name="r_arm_link_07_2_mass" value="1.50"/> <!--add 400g -->
   <xacro:property name="l_arm_link_01_mass" value="3.35"/>
   <xacro:property name="l_arm_link_02_mass" value="3.51"/>
@@ -49,5 +49,5 @@
   <xacro:property name="l_arm_link_07_mass" value="1.147"/>
   <xacro:property name="l_arm_link_07_1_mass" value="0.50"/>
-  <xacro:property name="l_arm_link_07_2_mass" value="0.65"/>
+  <xacro:property name="l_arm_link_07_2_mass" value="1.05"/> <!--add 400g -->
 <!-- link_inertia -->
   <xacro:property name="base_link_ixx" value="0.0"/>

Commit message: #20-2 slerp vel&acc
test

File: DualArm/dualarm_description/urdf/robot_parameter.xacro (robot description, xacro)
@@ -40,5 +40,5 @@
   <xacro:property name="r_arm_link_07_mass" value="1.60"/>
   <xacro:property name="r_arm_link_07_1_mass" value="0.50"/>
-  <xacro:property name="r_arm_link_07_2_mass" value="1.50"/> <!--add 400g -->
+  <xacro:property name="r_arm_link_07_2_mass" value="1.10"/>
   <xacro:property name="l_arm_link_01_mass" value="3.35"/>
   <xacro:property name="l_arm_link_02_mass" value="3.51"/>
@@ -49,5 +49,5 @@
   <xacro:property name="l_arm_link_07_mass" value="1.147"/>
   <xacro:property name="l_arm_link_07_1_mass" value="0.50"/>
-  <xacro:property name="l_arm_link_07_2_mass" value="1.05"/> <!--add 400g -->
+  <xacro:property name="l_arm_link_07_2_mass" value="0.65"/>
 <!-- link_inertia -->
   <xacro:property name="base_link_ixx" value="0.0"/>
