Commit message: #10 update minor bugs

File: DualArm/dualarm_description/urdf/dual_arm_ft.xacro (robot description, xacro)
@@ -1,4 +1,4 @@
 <?xml version="1.0"?>
-<robot name = "dualarm" xmlns:xacro="http://www.ros.org/wiki/xacro" >
+<robot name="dualarm" xmlns:xacro="http://www.ros.org/wiki/xacro" >
 	<xacro:include filename="$(find dualarm_description)/urdf/link_to_joint.xacro" />
 	<xacro:include filename="$(find dualarm_description)/urdf/robot_parameter.xacro" />
@@ -499,5 +499,5 @@
 				link="${r_arm_link_06_name}" />
 		<child
-				link="${r_arm_link_hand}" />
+				link="${r_arm_link_hand_1}" />
 		<dynamics damping="0.01" friction="0.01"/>
 	</joint>
@@ -515,25 +515,58 @@
 		</actuator>
 	</transmission>
-	<link name="${r_arm_link_hand}">
-		<inertial>
-			<mass value="${r_arm_link_07_mass}" />
-			<origin
-					rpy="0 0 0"
-					xyz="0.0099 0.0087 -0.126" />
-			<inertia
-					ixx="${r_arm_link_07_ixx}"
-					ixy="${r_arm_link_07_ixy}"
-					ixz="${r_arm_link_07_ixz}"
-					iyy="${r_arm_link_07_iyy}"
-					iyz="${r_arm_link_07_iyz}"
-					izz="${r_arm_link_07_izz}" />
-		</inertial>
-		<visual>
-			<origin
-					rpy="0 0 0"
-					xyz="0 0 0" />
-			<geometry>
-				<mesh
-						filename="package://dualarm_description/meshes/stl/r7.STL"
+	<link name="${r_arm_link_hand_1}">
+		<inertial>
+			<mass value="${r_arm_link_07_1_mass}" />
+			<origin
+					rpy="0 0 0"
+					xyz="0.0079 0.0 -0.0345" />
+			<inertia
+					ixx="${r_arm_link_07_1_ixx}"
+					ixy="${r_arm_link_07_1_ixy}"
+					ixz="${r_arm_link_07_1_ixz}"
+					iyy="${r_arm_link_07_1_iyy}"
+					iyz="${r_arm_link_07_1_iyz}"
+					izz="${r_arm_link_07_1_izz}" />
+		</inertial>
+		<visual>
+			<origin
+					rpy="0 0 0"
+					xyz="0 0 0" />
+			<geometry>
+				<mesh
+						filename="package://dualarm_description/meshes/stl/wrist_ft_R.STL"
+						scale="0.001 0.001 0.001"/>
+			</geometry>
+		</visual>
+	</link>
+	<joint name="ft_sensor_joint_R" type="fixed">
+		<parent link="${r_arm_link_hand_1}"/>
+		<child link="${r_arm_link_hand_2}"/>
+		<origin
+				rpy="0 0 0"
+				xyz="0 0 -0.057"/>
+		<limit effort="1000" velocity="100" lower="0" upper="0"/>
+	</joint>
+	<link name="${r_arm_link_hand_2}">
+		<inertial>
+			<mass value="${r_arm_link_07_2_mass}" />
+			<origin
+					rpy="0 0 0"
+					xyz="0.0112 0.0129 -0.1085" />
+			<inertia
+					ixx="${r_arm_link_07_2_ixx}"
+					ixy="${r_arm_link_07_2_ixy}"
+					ixz="${r_arm_link_07_2_ixz}"
+					iyy="${r_arm_link_07_2_iyy}"
+					iyz="${r_arm_link_07_2_iyz}"
+					izz="${r_arm_link_07_2_izz}" />
+		</inertial>
+		<visual>
+			<origin
+					rpy="0 0 0"
+					xyz="0 0 0" />
+			<geometry>
+				<mesh
+						filename="package://dualarm_description/meshes/stl/allegro_ft.STL"
 						scale="0.001 0.001 0.001"/>
 			</geometry>
@@ -542,7 +575,7 @@
 	<joint name="dualarm_R_end" type="fixed">
 		<origin
-				xyz="0 0 -0.167"
+				xyz="0 0 -0.110"
 				rpy="0 0 0"/>
-		<parent link="${r_arm_link_hand}"/>
+		<parent link="${r_arm_link_hand_2}"/>
 		<child link="dualarm_R_end_frame" />
 	</joint>
@@ -886,5 +919,5 @@
 				link="${l_arm_link_06_name}" />
 		<child
-				link="${l_arm_link_hand}" />
+				link="${l_arm_link_hand_1}" />
 		<dynamics damping="0.01" friction="0.01"/>
 	</joint>
@@ -902,25 +935,58 @@
 		</actuator>
 	</transmission>
-	<link name="${l_arm_link_hand}">
-		<inertial>
-			<mass value="${l_arm_link_07_mass}" />
-			<origin
-					rpy="0 0 0"
-					xyz="0.0188 -0.0157 -0.1202" />
-			<inertia
-					ixx="${l_arm_link_07_ixx}"
-					ixy="${l_arm_link_07_ixy}"
-					ixz="${l_arm_link_07_ixz}"
-					iyy="${l_arm_link_07_iyy}"
-					iyz="${l_arm_link_07_iyz}"
-					izz="${l_arm_link_07_izz}" />
-		</inertial>
-		<visual>
-			<origin
-					rpy="0 0 0"
-					xyz="0 0 0" />
-			<geometry>
-				<mesh
-						filename="package://dualarm_description/meshes/stl/l7.STL"
+	<link name="${l_arm_link_hand_1}">
+		<inertial>
+			<mass value="${l_arm_link_07_1_mass}" />
+			<origin
+					rpy="0 0 0"
+					xyz="0.0079 0.0 -0.0345" />
+			<inertia
+					ixx="${l_arm_link_07_1_ixx}"
+					ixy="${l_arm_link_07_1_ixy}"
+					ixz="${l_arm_link_07_1_ixz}"
+					iyy="${l_arm_link_07_1_iyy}"
+					iyz="${l_arm_link_07_1_iyz}"
+					izz="${l_arm_link_07_1_izz}" />
+		</inertial>
+		<visual>
+			<origin
+					rpy="0 0 0"
+					xyz="0 0 0" />
+			<geometry>
+				<mesh
+						filename="package://dualarm_description/meshes/stl/wrist_ft_L.STL"
+						scale="0.001 0.001 0.001"/>
+			</geometry>
+		</visual>
+	</link>
+	<joint name="ft_sensor_joint_L" type="fixed">
+		<parent link="${l_arm_link_hand_1}"/>
+		<child link="${l_arm_link_hand_2}"/>
+		<origin
+				rpy="0 0 0"
+				xyz="0 0 -0.057"/>
+		<limit effort="1000" velocity="100" lower="0" upper="0"/>
+	</joint>
+	<link name="${l_arm_link_hand_2}">
+		<inertial>
+			<mass value="${l_arm_link_07_2_mass}" />
+			<origin
+					rpy="0 0 0"
+					xyz="0.0282 -0.0237 -0.0862" />
+			<inertia
+					ixx="${l_arm_link_07_2_ixx}"
+					ixy="${l_arm_link_07_2_ixy}"
+					ixz="${l_arm_link_07_2_ixz}"
+					iyy="${l_arm_link_07_2_iyy}"
+					iyz="${l_arm_link_07_2_iyz}"
+					izz="${l_arm_link_07_2_izz}" />
+		</inertial>
+		<visual>
+			<origin
+					rpy="0 0 0"
+					xyz="0 0 0" />
+			<geometry>
+				<mesh
+						filename="package://dualarm_description/meshes/stl/lefthand_ft.STL"
 						scale="0.001 0.001 0.001"/>
 			</geometry>
@@ -929,7 +995,7 @@
 	<joint name="dualarm_L_end" type="fixed">
 		<origin
-				xyz="0 0 -0.167"
+				xyz="0 0 -0.110"
 				rpy="0 0 0"/>
-		<parent link="${l_arm_link_hand}"/>
+		<parent link="${l_arm_link_hand_2}"/>
 		<child link="dualarm_L_end_frame" />
 	</joint>

File: DualArm/dualarm_description/urdf/robot_parameter.xacro (robot description, xacro)
@@ -14,7 +14,7 @@
   <xacro:property name="r_arm_link_05_name" value="link_07" />
   <xacro:property name="r_arm_link_06_name" value="link_08" />
-  <xacro:property name="r_arm_link_hand" value="link_R_hand" />
-  <xacro:property name="r_arm_link_hand_1" value="link_R_hand_1" />
-  <xacro:property name="r_arm_link_hand_2" value="link_R_hand_2" />
+  <xacro:property name="r_arm_link_hand"    value="link_R_hand" />
+  <xacro:property name="r_arm_link_hand_1"  value="link_R_hand_1" />
+  <xacro:property name="r_arm_link_hand_2"  value="link_R_hand_2" />
 <!--left_arm-->
   <xacro:property name="l_arm_link_01_name" value="link_10" />
@@ -24,9 +24,9 @@
   <xacro:property name="l_arm_link_05_name" value="link_14" />
   <xacro:property name="l_arm_link_06_name" value="link_15" />
-  <xacro:property name="l_arm_link_hand" value="link_L_hand" />
-  <xacro:property name="l_arm_link_hand_1" value="link_L_hand_1" />
-  <xacro:property name="l_arm_link_hand_2" value="link_L_hand_2" />
+  <xacro:property name="l_arm_link_hand"    value="link_L_hand" />
+  <xacro:property name="l_arm_link_hand_1"  value="link_L_hand_1" />
+  <xacro:property name="l_arm_link_hand_2"  value="link_L_hand_2" />
 <!-- link_mass -->
-  <xacro:property name="base_link_mass" value="10.0"/>
+  <xacro:property name="base_link_mass"     value="10.0"/>
   <xacro:property name="waist_link_01_mass" value="11.91"/>
   <xacro:property name="waist_link_02_mass" value="10.901"/>

Commit message: #11 clik rqt update
RoM check

File: DualArm/dualarm_description/urdf/dual_arm_ft.xacro (robot description, xacro)
@@ -55,6 +55,6 @@
 		<limit
 				effort="300"
-				lower="-${M_PI}"
-				upper="${M_PI}"
+				lower="-${90.0*D2R}"
+				upper="${90.0*D2R}"
 				velocity="${2*M_PI}" />
 		<origin
@@ -109,6 +109,6 @@
 		<limit
 				effort="300"
-				lower="-${M_PI}"
-				upper="${M_PI}"
+				lower="-${90.0*D2R}"
+				upper="${90.0*D2R}"
 				velocity="${2*M_PI}" />
 		<origin
@@ -495,5 +495,5 @@
 		<origin
 				rpy="0 0 0"
-				xyz="0 0 -0.081" />
+				xyz="0 0 -0.091" />
 		<parent
 				link="${r_arm_link_06_name}" />
@@ -545,5 +545,5 @@
 		<origin
 				rpy="0 0 0"
-				xyz="0 0 -0.057"/>
+				xyz="0 0 -0.067"/>
 		<limit effort="1000" velocity="100" lower="0" upper="0"/>
 	</joint>
@@ -575,5 +575,5 @@
 	<joint name="dualarm_R_end" type="fixed">
 		<origin
-				xyz="0 0 -0.110"
+				xyz="0 0 -0.090"
 				rpy="0 0 0"/>
 		<parent link="${r_arm_link_hand_2}"/>
@@ -915,5 +915,5 @@
 		<origin
 				rpy="0 0 0"
-				xyz="0 0 -0.081" />
+				xyz="0 0 -0.091" />
 		<parent
 				link="${l_arm_link_06_name}" />
@@ -965,5 +965,5 @@
 		<origin
 				rpy="0 0 0"
-				xyz="0 0 -0.057"/>
+				xyz="0 0 -0.067"/>
 		<limit effort="1000" velocity="100" lower="0" upper="0"/>
 	</joint>
@@ -995,5 +995,5 @@
 	<joint name="dualarm_L_end" type="fixed">
 		<origin
-				xyz="0 0 -0.110"
+				xyz="0 0 -0.090"
 				rpy="0 0 0"/>
 		<parent link="${l_arm_link_hand_2}"/>

File: DualArm/dualarm_description/urdf/robot_parameter.xacro (robot description, xacro)
@@ -2,4 +2,5 @@
 <robot xmlns:xacro="http://www.ros.org/wiki/xacro">
   <xacro:property name="M_PI" value="3.141592"/>
+  <xacro:property name="D2R" value="57.2958"/>
 <!--base-->
   <xacro:property name="base_link_name" value="robot_base_link" />

Commit message: #12 clik ft_sensor& simulation update

File: DualArm/dualarm_description/urdf/dual_arm_ft.xacro (robot description, xacro)
@@ -569,7 +569,21 @@
 				<mesh
 						filename="package://dualarm_description/meshes/stl/allegro_ft.STL"
-						scale="0.001 0.001 0.001"/>
-			</geometry>
-		</visual>
+						scale="1 1 1"/>
+			</geometry>
+		</visual>
+		<collision name='collision'>
+			<geometry>
+				<mesh filename="package://dualarm_description/meshes/collision/allegro.dae"
+					  scale="1 1 1"/>
+			</geometry>
+			<surface>
+				<friction>
+					<ode>
+						<mu>100</mu>
+						<mu2>100</mu2>
+					</ode>
+				</friction>
+			</surface>
+		</collision>
 	</link>
 	<joint name="dualarm_R_end" type="fixed">
@@ -992,4 +1006,18 @@
 			</geometry>
 		</visual>
+		<collision name='collision'>
+			<geometry>
+				<mesh filename="package://dualarm_description/meshes/collision/lefthand_ft.dae"
+				scale="0.001 0.001 0.001"/>
+			</geometry>
+			<surface>
+				<friction>
+					<ode>
+						<mu>100</mu>
+						<mu2>100</mu2>
+					</ode>
+				</friction>
+			</surface>
+		</collision>
 	</link>
 	<joint name="dualarm_L_end" type="fixed">

Commit message: #17 task trajectory
5th trajectory

File: DualArm/dualarm_description/urdf/dual_arm_ft.xacro (robot description, xacro)
@@ -572,5 +572,5 @@
 			</geometry>
 		</visual>
-		<collision name='collision'>
+		<!--<collision name='collision'>
 			<geometry>
 				<mesh filename="package://dualarm_description/meshes/collision/allegro.dae"
@@ -585,5 +585,5 @@
 				</friction>
 			</surface>
-		</collision>
+		</collision>-->
 	</link>
 	<joint name="dualarm_R_end" type="fixed">
@@ -1006,5 +1006,5 @@
 			</geometry>
 		</visual>
-		<collision name='collision'>
+		<!--<collision name='collision'>
 			<geometry>
 				<mesh filename="package://dualarm_description/meshes/collision/lefthand_ft.dae"
@@ -1019,5 +1019,5 @@
 				</friction>
 			</surface>
-		</collision>
+		</collision> -->
 	</link>
 	<joint name="dualarm_L_end" type="fixed">

Commit message: #22 PID control + friction compensation (joint space)

File: DualArm/dualarm_description/urdf/dual_arm_ft.xacro (robot description, xacro)
@@ -65,5 +65,5 @@
 		<child
 				link="${waist_link_01_name}" />
-		<dynamics damping="0.01" friction="0.01"/>
+		<dynamics damping="1" friction="3"/>0
 	</joint>
 	<transmission
@@ -119,5 +119,5 @@
 		<child
 				link="${waist_link_02_name}" />
-		<dynamics damping="0.01" friction="0.01"/>
+		<dynamics damping="1" friction="4"/>
 	</joint>
 	<transmission
@@ -176,5 +176,5 @@
 		<child
 				link="${r_arm_link_01_name}" />
-		<dynamics damping="0.01" friction="0.01"/>
+		<dynamics damping="1" friction="2"/>
 	</joint>
 	<transmission
@@ -230,5 +230,5 @@
 		<child
 				link="${r_arm_link_02_name}" />
-		<dynamics damping="0.01" friction="0.01"/>
+		<dynamics damping="1" friction="2"/>
 	</joint>
 	<transmission
@@ -284,5 +284,5 @@
 		<child
 				link="${r_arm_link_03_name}" />
-		<dynamics damping="0.01" friction="0.01"/>
+		<dynamics damping="1" friction="2"/>
 	</joint>
 	<transmission
@@ -338,5 +338,5 @@
 		<child
 				link="${r_arm_link_04_name}" />
-		<dynamics damping="0.01" friction="0.01"/>
+		<dynamics damping="1" friction="2.5"/>
 	</joint>
 	<transmission
@@ -392,5 +392,5 @@
 		<child
 				link="${r_arm_link_05_name}" />
-		<dynamics damping="0.01" friction="0.01"/>
+		<dynamics damping="1" friction="2"/>
 	</joint>
 	<transmission
@@ -446,5 +446,5 @@
 		<child
 				link="${r_arm_link_06_name}" />
-		<dynamics damping="0.01" friction="0.01"/>
+		<dynamics damping="1" friction="2.8"/>
 	</joint>
 	<transmission
@@ -500,5 +500,5 @@
 		<child
 				link="${r_arm_link_hand_1}" />
-		<dynamics damping="0.01" friction="0.01"/>
+		<dynamics damping="1" friction="2.8"/>
 	</joint>
 	<transmission
@@ -610,5 +610,5 @@
 		<child
 				link="${l_arm_link_01_name}" />
-		<dynamics damping="0.01" friction="0.01"/>
+		<dynamics damping="1" friction="2"/>
 	</joint>
 	<transmission
@@ -664,5 +664,5 @@
 		<child
 				link="${l_arm_link_02_name}" />
-		<dynamics damping="0.01" friction="0.01"/>
+		<dynamics damping="1" friction="2"/>
 	</joint>
 	<transmission
@@ -718,5 +718,5 @@
 		<child
 				link="${l_arm_link_03_name}" />
-		<dynamics damping="0.01" friction="0.01"/>
+		<dynamics damping="1" friction="2"/>
 	</joint>
 	<transmission
@@ -772,5 +772,5 @@
 		<child
 				link="${l_arm_link_04_name}" />
-		<dynamics damping="0.01" friction="0.01"/>
+		<dynamics damping="1" friction="2.5"/>
 	</joint>
 	<transmission
@@ -826,5 +826,5 @@
 		<child
 				link="${l_arm_link_05_name}" />
-		<dynamics damping="0.01" friction="0.01"/>
+		<dynamics damping="1" friction="2"/>
 	</joint>
 	<transmission
@@ -880,5 +880,5 @@
 		<child
 				link="${l_arm_link_06_name}" />
-		<dynamics damping="0.01" friction="0.01"/>
+		<dynamics damping="1" friction="2.8"/>
 	</joint>
 	<transmission
@@ -934,5 +934,5 @@
 		<child
 				link="${l_arm_link_hand_1}" />
-		<dynamics damping="0.01" friction="0.01"/>
+		<dynamics damping="1" friction="2.8"/>
 	</joint>
 	<transmission

Commit message: #23 data plot setting

File: DualArm/dualarm_description/urdf/dual_arm_ft.xacro (robot description, xacro)
@@ -65,5 +65,5 @@
 		<child
 				link="${waist_link_01_name}" />
-		<dynamics damping="1" friction="3"/>0
+		<dynamics damping="0.01" friction="0.1"/>0
 	</joint>
 	<transmission
@@ -119,5 +119,5 @@
 		<child
 				link="${waist_link_02_name}" />
-		<dynamics damping="1" friction="4"/>
+		<dynamics damping="1" friction="1"/>
 	</joint>
 	<transmission
@@ -176,5 +176,5 @@
 		<child
 				link="${r_arm_link_01_name}" />
-		<dynamics damping="1" friction="2"/>
+		<dynamics damping="0.01" friction="0.1"/>
 	</joint>
 	<transmission
@@ -230,5 +230,5 @@
 		<child
 				link="${r_arm_link_02_name}" />
-		<dynamics damping="1" friction="2"/>
+		<dynamics damping="0.01" friction="0.1"/>
 	</joint>
 	<transmission
@@ -284,5 +284,5 @@
 		<child
 				link="${r_arm_link_03_name}" />
-		<dynamics damping="1" friction="2"/>
+		<dynamics damping="0.01" friction="0.1"/>
 	</joint>
 	<transmission
@@ -338,5 +338,5 @@
 		<child
 				link="${r_arm_link_04_name}" />
-		<dynamics damping="1" friction="2.5"/>
+		<dynamics damping="0.01" friction="0.1"/>
 	</joint>
 	<transmission
@@ -392,5 +392,5 @@
 		<child
 				link="${r_arm_link_05_name}" />
-		<dynamics damping="1" friction="2"/>
+		<dynamics damping="0.01" friction="0.1"/>
 	</joint>
 	<transmission
@@ -446,5 +446,5 @@
 		<child
 				link="${r_arm_link_06_name}" />
-		<dynamics damping="1" friction="2.8"/>
+		<dynamics damping="0.01" friction="0.1"/>
 	</joint>
 	<transmission
@@ -500,5 +500,5 @@
 		<child
 				link="${r_arm_link_hand_1}" />
-		<dynamics damping="1" friction="2.8"/>
+		<dynamics damping="0.01" friction="0.1"/>
 	</joint>
 	<transmission
@@ -610,5 +610,5 @@
 		<child
 				link="${l_arm_link_01_name}" />
-		<dynamics damping="1" friction="2"/>
+		<dynamics damping="0.01" friction="0.1"/>
 	</joint>
 	<transmission
@@ -664,5 +664,5 @@
 		<child
 				link="${l_arm_link_02_name}" />
-		<dynamics damping="1" friction="2"/>
+		<dynamics damping="0.01" friction="0.1"/>
 	</joint>
 	<transmission
@@ -718,5 +718,5 @@
 		<child
 				link="${l_arm_link_03_name}" />
-		<dynamics damping="1" friction="2"/>
+		<dynamics damping="0.01" friction="0.1"/>
 	</joint>
 	<transmission
@@ -772,5 +772,5 @@
 		<child
 				link="${l_arm_link_04_name}" />
-		<dynamics damping="1" friction="2.5"/>
+		<dynamics damping="0.01" friction="0.1"/>
 	</joint>
 	<transmission
@@ -826,5 +826,5 @@
 		<child
 				link="${l_arm_link_05_name}" />
-		<dynamics damping="1" friction="2"/>
+		<dynamics damping="0.01" friction="0.1"/>
 	</joint>
 	<transmission
@@ -880,5 +880,5 @@
 		<child
 				link="${l_arm_link_06_name}" />
-		<dynamics damping="1" friction="2.8"/>
+		<dynamics damping="0.01" friction="0.1"/>
 	</joint>
 	<transmission
@@ -924,6 +924,6 @@
 		<limit
 				effort="300"
-				lower="-0.7854"
-				upper="0.7854"
+				lower="-1.5708"
+				upper="1.5708"
 				velocity="${M_PI}" />
 		<origin
@@ -934,5 +934,5 @@
 		<child
 				link="${l_arm_link_hand_1}" />
-		<dynamics damping="1" friction="2.8"/>
+		<dynamics damping="0.01" friction="0.1"/>
 	</joint>
 	<transmission

Commit message: #24 vive_tracker for simulation

File: DualArm/dualarm_description/urdf/dual_arm_ft.xacro (robot description, xacro)
@@ -65,5 +65,5 @@
 		<child
 				link="${waist_link_01_name}" />
-		<dynamics damping="0.01" friction="0.1"/>0
+		<dynamics damping="0.01" friction="1"/>0
 	</joint>
 	<transmission
@@ -176,5 +176,5 @@
 		<child
 				link="${r_arm_link_01_name}" />
-		<dynamics damping="0.01" friction="0.1"/>
+		<dynamics damping="0.01" friction="1"/>
 	</joint>
 	<transmission
@@ -230,5 +230,5 @@
 		<child
 				link="${r_arm_link_02_name}" />
-		<dynamics damping="0.01" friction="0.1"/>
+		<dynamics damping="0.01" friction="1"/>
 	</joint>
 	<transmission
@@ -284,5 +284,5 @@
 		<child
 				link="${r_arm_link_03_name}" />
-		<dynamics damping="0.01" friction="0.1"/>
+		<dynamics damping="0.01" friction="1"/>
 	</joint>
 	<transmission
@@ -338,5 +338,5 @@
 		<child
 				link="${r_arm_link_04_name}" />
-		<dynamics damping="0.01" friction="0.1"/>
+		<dynamics damping="0.01" friction="1"/>
 	</joint>
 	<transmission
@@ -392,5 +392,5 @@
 		<child
 				link="${r_arm_link_05_name}" />
-		<dynamics damping="0.01" friction="0.1"/>
+		<dynamics damping="0.01" friction="1"/>
 	</joint>
 	<transmission
@@ -436,6 +436,6 @@
 		<limit
 				effort="300"
-				lower="-0.7854"
-				upper="0.7854"
+				lower="-2.037"
+				upper="2.037"
 				velocity="${2*M_PI}" />
 		<origin
@@ -446,5 +446,5 @@
 		<child
 				link="${r_arm_link_06_name}" />
-		<dynamics damping="0.01" friction="0.1"/>
+		<dynamics damping="0.01" friction="1"/>
 	</joint>
 	<transmission
@@ -500,5 +500,5 @@
 		<child
 				link="${r_arm_link_hand_1}" />
-		<dynamics damping="0.01" friction="0.1"/>
+		<dynamics damping="0.01" friction="1"/>
 	</joint>
 	<transmission
@@ -610,5 +610,5 @@
 		<child
 				link="${l_arm_link_01_name}" />
-		<dynamics damping="0.01" friction="0.1"/>
+		<dynamics damping="0.01" friction="1"/>
 	</joint>
 	<transmission
@@ -664,5 +664,5 @@
 		<child
 				link="${l_arm_link_02_name}" />
-		<dynamics damping="0.01" friction="0.1"/>
+		<dynamics damping="0.01" friction="1"/>
 	</joint>
 	<transmission
@@ -718,5 +718,5 @@
 		<child
 				link="${l_arm_link_03_name}" />
-		<dynamics damping="0.01" friction="0.1"/>
+		<dynamics damping="0.01" friction="1"/>
 	</joint>
 	<transmission
@@ -772,5 +772,5 @@
 		<child
 				link="${l_arm_link_04_name}" />
-		<dynamics damping="0.01" friction="0.1"/>
+		<dynamics damping="0.01" friction="1"/>
 	</joint>
 	<transmission
@@ -826,5 +826,5 @@
 		<child
 				link="${l_arm_link_05_name}" />
-		<dynamics damping="0.01" friction="0.1"/>
+		<dynamics damping="0.01" friction="1"/>
 	</joint>
 	<transmission
@@ -870,6 +870,6 @@
 		<limit
 				effort="300"
-				lower="-${M_PI}"
-				upper="${M_PI}"
+				lower="-2.037"
+				upper="2.037"
 				velocity="${M_PI}" />
 		<origin
@@ -880,5 +880,5 @@
 		<child
 				link="${l_arm_link_06_name}" />
-		<dynamics damping="0.01" friction="0.1"/>
+		<dynamics damping="0.01" friction="1"/>
 	</joint>
 	<transmission
@@ -934,5 +934,5 @@
 		<child
 				link="${l_arm_link_hand_1}" />
-		<dynamics damping="0.01" friction="0.1"/>
+		<dynamics damping="0.01" friction="1"/>
 	</joint>
 	<transmission

Commit message: #27 depense

File: DualArm/dualarm_description/urdf/dual_arm_ft.xacro (robot description, xacro)
@@ -572,18 +572,22 @@
 			</geometry>
 		</visual>
-		<!--<collision name='collision'>
-			<geometry>
-				<mesh filename="package://dualarm_description/meshes/collision/allegro.dae"
-					  scale="1 1 1"/>
+ 		<collision name='collision'>
+ 			<origin
+					rpy="1.5707 0 0"
+					xyz="0 0 -0.1" />
+			<geometry>
+				<!--<mesh filename="package://dualarm_description/meshes/collision/lefthand_ft.dae"
+				scale="0.001 0.001 0.001"/>-->
+				<box size="0.0996 0.16 0.0491"/>
 			</geometry>
 			<surface>
 				<friction>
 					<ode>
-						<mu>100</mu>
-						<mu2>100</mu2>
-					</ode>
+						<mu>1</mu>
+ 						<mu2>1</mu2>
+ 					</ode>
 				</friction>
 			</surface>
-		</collision>-->
+		</collision>
 	</link>
 	<joint name="dualarm_R_end" type="fixed">
@@ -997,5 +1001,5 @@
 		</inertial>
 		<visual>
-			<origin
+		<origin
 					rpy="0 0 0"
 					xyz="0 0 0" />
@@ -1006,18 +1010,22 @@
 			</geometry>
 		</visual>
-		<!--<collision name='collision'>
-			<geometry>
-				<mesh filename="package://dualarm_description/meshes/collision/lefthand_ft.dae"
-				scale="0.001 0.001 0.001"/>
+ 		<collision name='collision'>
+			<origin
+					rpy="1.5707 0 0"
+					xyz="0 -0.01 -0.1" />
+			<geometry>
+				<!--<mesh filename="package://dualarm_description/meshes/collision/lefthand_ft.dae"
+				scale="0.001 0.001 0.001"/>-->
+				<box size="0.0996 0.16 0.0491"/>
 			</geometry>
 			<surface>
 				<friction>
 					<ode>
-						<mu>100</mu>
-						<mu2>100</mu2>
+						<mu>1</mu>
+ 						<mu2>1</mu2>
 					</ode>
 				</friction>
 			</surface>
-		</collision> -->
+		</collision>
 	</link>
 	<joint name="dualarm_L_end" type="fixed">
